Commit message: :bug: fixed tugger tree

File: urdf/glr_tugger.xacro (robot description, xacro)
@@ -18,15 +18,8 @@
     </inertial>
   </xacro:macro>
-  <!--Robot description  -->
-  <link name="base_link"/>
-  <!-- Robot Footprint -->
+  <!-- Robot Footprint (on the ground) -->
   <link name="base_footprint"/>
-  <joint name="base_joint" type="fixed">
-    <parent link="base_link"/>
-    <child link="base_footprint"/>
-    <origin xyz="0 0 0" rpy="0 0 0"/>
-  </joint>
-  <!-- Tugger -->
-  <link name="chassibigga">
+  <!-- Tugger Main Body (base_link) -->
+  <link name="base_link">
     <origin xyz="0 0 0" rpy="0 0 0" />
     <inertial>
@@ -51,7 +44,7 @@
     </collision>
   </link>
-  <joint name="base_chassi_joint" type="fixed">
-    <parent link="base_link"/>
-    <child link="chassibigga"/>
+  <joint name="base_joint" type="fixed">
+    <parent link="base_footprint"/>
+    <child link="base_link"/>
     <origin xyz="0 0 ${wheel_radius}" rpy="0 0 0"/>
   </joint>
@@ -81,5 +74,5 @@
   <joint name="left_wheel_joint" type="continuous">
     <origin xyz="0.25 0 0" rpy="0 0 0"/>
-    <parent link="chassibigga"/>
+    <parent link="base_link"/>
     <child link="left_wheel"/>
     <axis xyz="1 0 0"/>
@@ -111,5 +104,5 @@
   <joint name="right_wheel_joint" type="continuous">
     <origin xyz="-0.25 0 0" rpy="0 0 0"/>
-    <parent link="chassibigga"/>
+    <parent link="base_link"/>
     <child link="right_wheel"/>
     <axis xyz="1 0 0"/>
@@ -144,5 +137,5 @@
   <joint name="hitch_joint" type="fixed">
     <origin xyz="0 0.35 0.14260" rpy="0 0 0"/>
-    <parent link="chassibigga"/>
+    <parent link="base_link"/>
     <child link="hitch_link"/>
   </joint>
@@ -171,5 +164,5 @@
   </link>
   <joint name="lidar_joint" type="fixed">
-    <parent link="chassibigga"/>
+    <parent link="base_link"/>
     <child link="lidar_link"/>
     <origin xyz="0 -0.25 0.34" rpy="0 0 0"/>

File: urdf/glr_tugger_gazebo.xacro (robot description, xacro)
@@ -4,5 +4,5 @@
   <!-- TUGGER GAZEBO MATERIAL DEFINITIONS -->
   <!-- ============================================ -->
-  <gazebo reference="chassibigga">
+  <gazebo reference="base_link">
     <material>Gazebo/Orange</material>
   </gazebo>
