Commit message: :sparkles: removed cameras and added generic lidar instead of velodyne

File: urdf/glr.xacro (robot description, xacro)
@@ -1510,86 +1510,68 @@
       k_velocity="0" />
   </joint>
-  <!-- sensor -->
-  <xacro:property name="camera_link" value="0.05" />
-  <!-- Camera -->
-  <link name="camera_link">
+  <!-- Generic LiDAR -->
+  <link name="lidar_link">
+    <inertial>
+      <origin xyz="0 0 0" rpy="0 0 0"/>
+      <mass value="0.5"/>
+      <inertia ixx="0.001" ixy="0" ixz="0" iyy="0.001" iyz="0" izz="0.001"/>
+    </inertial>
+    <visual>
+      <origin xyz="0 0 0" rpy="0 0 0"/>
+      <geometry>
+        <cylinder radius="0.05" length="0.07"/>
+      </geometry>
+      <material name="lidar_material">
+        <color rgba="0.2 0.2 0.2 1"/>
+      </material>
+    </visual>
     <collision>
       <origin xyz="0 0 0" rpy="0 0 0"/>
       <geometry>
-    <box size="${camera_link} ${camera_link} ${camera_link}"/>
+        <cylinder radius="0.05" length="0.07"/>
       </geometry>
     </collision>
-    <visual>
-      <origin xyz="0 0 0" rpy="0 0 0"/>
-      <geometry>
-    <box size="${camera_link} ${camera_link} ${camera_link}"/>
-      </geometry>
-    </visual>
-    <inertial>
-      <mass value="1e-5" />
-      <origin xyz="0 0 0" rpy="0 0 0"/>
-      <inertia ixx="1e-6" ixy="0" ixz="0" iyy="1e-6" iyz="0" izz="1e-6" />
-    </inertial>
-  </link>
-  <joint name="camera_joint" type="fixed">
-    <axis xyz="0 1 0" />
-    <origin xyz="0 -1.6 0.6" rpy="0 0 -1.57"/>
+  </link>
+  <joint name="lidar_joint" type="fixed">
     <parent link="chassibigga"/>
-    <child link="camera_link"/>
-  </joint>
-  <!-- camera -->
-  <gazebo reference="camera_link">
-    <sensor type="camera" name="camera">
-      <update_rate>40.0</update_rate>
-      <camera name="head">
-        <horizontal_fov>1.3962634</horizontal_fov>
-        <image>
-          <width>800</width>
-          <height>800</height>
-          <format>R8G8B8</format>
-        </image>
-        <clip>
-          <near>0.02</near>
-          <far>300</far>
-        </clip>
+    <child link="lidar_link"/>
+    <origin xyz="0 -1.7 0.4" rpy="0 0 0"/>
+  </joint>
+  <gazebo reference="lidar_link">
+    <material>Gazebo/DarkGrey</material>
+    <sensor type="ray" name="lidar_sensor">
+      <pose>0 0 0 0 0 0</pose>
+      <visualize>true</visualize>
+      <update_rate>10</update_rate>
+      <ray>
+        <scan>
+          <horizontal>
+            <samples>360</samples>
+            <resolution>1</resolution>
+            <min_angle>-3.14159</min_angle>
+            <max_angle>3.14159</max_angle>
+          </horizontal>
+        </scan>
+        <range>
+          <min>0.1</min>
+          <max>30.0</max>
+          <resolution>0.01</resolution>
+        </range>
         <noise>
           <type>gaussian</type>
-          <!-- Noise is sampled independently per pixel on each frame.
-               That pixel's noise value is added to each of its color
-               channels, which at that point lie in the range [0,1]. -->
           <mean>0.0</mean>
-          <stddev>0.007</stddev>
+          <stddev>0.01</stddev>
         </noise>
-      </camera>
-      <plugin name="camera_controller" filename="libgazebo_ros_camera.so">
+      </ray>
+      <plugin name="gazebo_ros_lidar" filename="libgazebo_ros_ray_sensor.so">
         <ros>
-            <namespace>/glr_description</namespace>
-            <!-- <remapping>/glr_description/imu_plugin/out:=/glr_description/imu</remapping> -->
+          <namespace>/glr_description</namespace>
+          <remapping>~/out:=scan</remapping>
         </ros>
-        <alwaysOn>true</alwaysOn>
-        <updateRate>0.0</updateRate>
-        <cameraName>rrbot/camera1</cameraName>
-        <imageTopicName>image_raw</imageTopicName>
-        <cameraInfoTopicName>camera_info</cameraInfoTopicName>
-        <frameName>camera_link</frameName>
-        <hackBaseline>0.07</hackBaseline>
-        <distortionK1>0.0</distortionK1>
-        <distortionK2>0.0</distortionK2>
-        <distortionK3>0.0</distortionK3>
-        <distortionT1>0.0</distortionT1>
-        <distortionT2>0.0</distortionT2>
+        <output_type>sensor_msgs/LaserScan</output_type>
+        <frame_name>lidar_link</frame_name>
       </plugin>
     </sensor>
-    <material>Gazebo/Red</material>
-  </gazebo>
-  <!-- velodyne -->
-  <xacro:arg name="gpu" default="false"/>
-  <xacro:property name="gpu" value="$(arg gpu)" />
-  <xacro:arg name="organize_cloud" default="false"/>
-  <xacro:property name="organize_cloud" value="$(arg organize_cloud)" />
-  <xacro:include filename="VLP-16.urdf.xacro"/>
-  <xacro:VLP-16 parent="chassibigga" name="velodyne" topic="points2" organize_cloud="${organize_cloud}" hz="10" samples="440" gpu="${gpu}" min_angle="-3.1415926535897931" max_angle="0.0">
-    <origin xyz="0 -1.7 0.4" rpy="0 0 0" />
-  </xacro:VLP-16>
+  </gazebo>
   <!-- modelo da IMU -->
   <link name="imu_link">
@@ -1636,82 +1618,3 @@
     </sensor>
   </gazebo>
-  <!-- sensor -->
-  <xacro:property name="camera2_link" value="0.05" />
-  <!-- Camera -->
-  <link name="camera2_link">
-    <collision>
-      <origin xyz="0 0 0" rpy="0 0 0"/>
-      <geometry>
-        <box size="${camera2_link} ${camera2_link} ${camera2_link}"/>
-      </geometry>
-    </collision>
-    <visual>
-      <origin xyz="0 0 0" rpy="0 0 0"/>
-      <geometry>
-        <box size="${camera2_link} ${camera2_link} ${camera2_link}"/>
-      </geometry>
-    </visual>
-    <inertial>
-      <mass value="1e-5" />
-      <origin xyz="0 0 0" rpy="0 0 0"/>
-      <inertia ixx="1e-6" ixy="0" ixz="0" iyy="1e-6" iyz="0" izz="1e-6" />
-    </inertial>
-  </link>
-  <joint name="camera2_joint" type="fixed">
-    <axis xyz="0 1 0" />
-    <origin xyz="0 0 0.5" rpy="0 0 -3.14"/>
-    <parent link="chassi"/>
-    <child link="camera2_link"/>
-  </joint>
-  <!-- camera -->
-  <gazebo reference="camera2_link">
-    <sensor type="camera" name="camera2">
-      <update_rate>40.0</update_rate>
-      <camera name="head">
-        <horizontal_fov>1.3962634</horizontal_fov>
-        <image>
-          <width>800</width>
-          <height>800</height>
-          <format>R8G8B8</format>
-        </image>
-        <clip>
-          <near>0.02</near>
-          <far>300</far>
-        </clip>
-        <noise>
-          <type>gaussian</type>
-          <!-- Noise is sampled independently per pixel on each frame.
-               That pixel's noise value is added to each of its color
-               channels, which at that point lie in the range [0,1]. -->
-          <mean>0.0</mean>
-          <stddev>0.007</stddev>
-        </noise>
-      </camera>
-      <plugin name="camera2_controller" filename="libgazebo_ros_camera.so">
-        <ros>
-            <namespace>/glr_description</namespace>
-            <!-- <remapping>/glr_description/imu_plugin/out:=/glr_description/imu</remapping> -->
-        </ros>
-        <alwaysOn>true</alwaysOn>
-        <updateRate>0.0</updateRate>
-        <cameraName>rrbot/camera21</cameraName>
-        <imageTopicName>image_raw2</imageTopicName>
-        <cameraInfoTopicName>camera2_info</cameraInfoTopicName>
-        <frameName>camera2_link</frameName>
-        <hackBaseline>0.07</hackBaseline>
-        <distortionK1>0.0</distortionK1>
-        <distortionK2>0.0</distortionK2>
-        <distortionK3>0.0</distortionK3>
-        <distortionT1>0.0</distortionT1>
-        <distortionT2>0.0</distortionT2>
-      </plugin>
-    </sensor>
-    <material>Gazebo/Red</material>
-  </gazebo>
-    <!-- <joint name="camera_joint" type="fixed">
-    <axis xyz="0 1 0" />
-    <origin xyz="0 -1.6 0.5" rpy="0 0 -1.57"/>
-    <parent link="chassibigga"/>
-    <child link="camera_link"/>
-  </joint> -->
 </robot>

Commit message: :zap: removed some joints

File: urdf/glr.xacro (robot description, xacro)
@@ -23,5 +23,5 @@
     <parent link="base_link"/>
     <child link="base_footprint"/>
-    <origin xyz="0 0 0" rpy="0 0 -1.5708"/> <!-- Adjusted orientation by 90 degrees (1.5708 radians) -->
+    <origin xyz="0 0 0" rpy="0 0 0"/>
   </joint>
   <!-- Tugger -->
@@ -32,5 +32,5 @@
     <inertial>
       <origin
-        xyz="0. -0.81 0."
+        xyz="0 0 0.38"
         rpy="0 0 0" />
       <mass
@@ -40,5 +40,5 @@
     <visual>
       <origin
-        xyz="0 -0.8 0.38"
+        xyz="0 0 0.38"
         rpy="0 0 0" />
       <geometry>
@@ -53,5 +53,5 @@
     <collision>
       <origin
-        xyz="0 -0.8 0.38"
+        xyz="0 0 0.38"
         rpy="0 0 0" />
       <geometry>
@@ -67,135 +67,271 @@
     <child link="chassibigga"/>
   </joint>
-  <link name="volantebigga">
-    <inertial>
-      <origin
-        xyz="0.0017469 -0.08522 0.13505"
-        rpy="0 0 0" />
-      <mass
-        value="2.496" />
-      <inertia
-        ixx="5.5"
-        ixy="0.0"
-        ixz="0.0"
-        iyy="5.5"
-        iyz="0.0"
-        izz="5.5" />
-    </inertial>
-    <!-- <visual>
-      <origin
-        xyz="0 0 0"
-        rpy="0 0 0" />
-      <geometry>
-        <mesh
-          filename="package://glr_description/models/volantebigga.STL" />
-      </geometry>
-      <material
-        name="">
-        <color
-          rgba="0.64706 0.61961 0.58824 1" />
-      </material>
-    </visual> -->
-  </link>
-  <gazebo reference="volantebigga">
-    <material>Gazebo/Orange</material>
-  </gazebo>
-  <joint name="eixovolantebigga"
-    type="fixed">
-    <origin
-      xyz="0 -1.3437 0.19438"
-      rpy="-0.13255 0 0" />
-    <parent link="chassibigga" />
-    <child link="volantebigga" />
-  </joint>
-  <link name="rodavolantebigga">
-    <inertial>
-      <origin
-        xyz="-0.00 0 0"
-        rpy="0 0 0" />
-      <mass
-        value="12" />
+  <!-- ============================================ -->
+  <!-- DIFFERENTIAL DRIVE WHEELS (Center - Traction) -->
+  <!-- ============================================ -->
+  <!-- Left Traction Wheel -->
+  <link name="left_wheel">
+    <inertial>
+      <origin xyz="0 0 0" rpy="0 0 0"/>
+      <mass value="12"/>
       <xacro:sphere_inertia m="12" r="0.14260"/>
     </inertial>
     <visual>
-      <origin
-        xyz="0.0 0 0"
-        rpy="0 1.5708 0" />
-      <geometry>
-        <cylinder radius="0.14260" length="0.16"/>
-      </geometry>
-      <material
-        name="">
-        <color
-          rgba="0.29804 0.29804 0.29804 1" />
-      </material>
-    </visual>
-    <collision>
-      <origin
-        xyz="-0.0 0 0"
-        rpy="0 1.5708 0" />
-      <geometry>
-        <sphere radius="0.14260"/>
-      </geometry>
-    </collision>
-  </link>
-  <gazebo reference="rodavolantebigga">
+      <origin xyz="0 0 0" rpy="1.5708 0 0"/>
+      <geometry>
+        <cylinder radius="0.14260" length="0.08"/>
+      </geometry>
+      <material name="wheel_material">
+        <color rgba="0.29804 0.29804 0.29804 1"/>
+      </material>
+    </visual>
+    <collision>
+      <origin xyz="0 0 0" rpy="1.5708 0 0"/>
+      <geometry>
+        <cylinder radius="0.14260" length="0.08"/>
+      </geometry>
+    </collision>
+  </link>
+  <gazebo reference="left_wheel">
     <material>Gazebo/Black</material>
-  </gazebo>
-  <link name="rodavolantebigga_uni">
-    <inertial>
-      <origin
-        xyz="-0. 0 0"
-        rpy="0 0 0" />
-      <mass
-        value="12" />
+    <mu1>1.0</mu1>
+    <mu2>1.0</mu2>
+  </gazebo>
+  <joint name="left_wheel_joint" type="continuous">
+    <origin xyz="0.5 0 0" rpy="0 0 0"/>
+    <parent link="chassibigga"/>
+    <child link="left_wheel"/>
+    <axis xyz="1 0 0"/>
+    <dynamics damping="0.1" friction="0.1"/>
+  </joint>
+  <!-- Right Traction Wheel -->
+  <link name="right_wheel">
+    <inertial>
+      <origin xyz="0 0 0" rpy="0 0 0"/>
+      <mass value="12"/>
       <xacro:sphere_inertia m="12" r="0.14260"/>
     </inertial>
-  </link>
-  <joint name="eixorodavolantebigga_steer"
-    type="revolute">
-    <origin
-      xyz="0.00 -0.024481 -0.38947"
-      rpy="0 0 0" />
-    <parent link="volantebigga" />
-    <child link="rodavolantebigga_uni" />
-    <axis
-      xyz="0 0 1" />
-    <limit
-      lower="-0.7"
-      upper="0.7"
-      effort="100"
-      velocity="1" />
-    <calibration
-      rising="0"
-      falling="0" />
-    <dynamics
-      damping="0"
-      friction="1.0" />
-    <safety_controller
-      soft_upper="0"
-      soft_lower="0"
-      k_position="0"
-      k_velocity="0" />
-  </joint>
-  <joint name="eixorodavolantebigga"
-    type="continuous">
-    <origin
-      xyz="0. -0. -0."
-      rpy="0 0 0" />
-    <parent link="rodavolantebigga_uni" />
-    <child link="rodavolantebigga" />
-    <axis
-      xyz="1 0 0" />
-    <calibration
-      rising="0"
-      falling="0" />
-    <dynamics
-      damping="0"
-      friction="10.0" />
-    <safety_controller
-      soft_upper="0"
-      soft_lower="0"
-      k_position="0"
-      k_velocity="0" />
+    <visual>
+      <origin xyz="0 0 0" rpy="1.5708 0 0"/>
+      <geometry>
+        <cylinder radius="0.14260" length="0.08"/>
+      </geometry>
+      <material name="wheel_material">
+        <color rgba="0.29804 0.29804 0.29804 1"/>
+      </material>
+    </visual>
+    <collision>
+      <origin xyz="0 0 0" rpy="1.5708 0 0"/>
+      <geometry>
+        <cylinder radius="0.14260" length="0.08"/>
+      </geometry>
+    </collision>
+  </link>
+  <gazebo reference="right_wheel">
+    <material>Gazebo/Black</material>
+    <mu1>1.0</mu1>
+    <mu2>1.0</mu2>
+  </gazebo>
+  <joint name="right_wheel_joint" type="continuous">
+    <origin xyz="-0.5 0 0" rpy="0 0 0"/>
+    <parent link="chassibigga"/>
+    <child link="right_wheel"/>
+    <axis xyz="1 0 0"/>
+    <dynamics damping="0.1" friction="0.1"/>
+  </joint>
+  <!-- ============================================ -->
+  <!-- CASTER WHEELS (Front - 2 wheels) -->
+  <!-- ============================================ -->
+  <!-- Front Left Caster -->
+  <link name="front_left_caster">
+    <inertial>
+      <origin xyz="0 0 0" rpy="0 0 0"/>
+      <mass value="0.5"/>
+      <xacro:sphere_inertia m="0.5" r="0.05"/>
+    </inertial>
+    <visual>
+      <origin xyz="0 0 0" rpy="0 0 0"/>
+      <geometry>
+        <sphere radius="0.05"/>
+      </geometry>
+      <material name="caster_material">
+        <color rgba="0.5 0.5 0.5 1"/>
+      </material>
+    </visual>
+    <collision>
+      <origin xyz="0 0 0" rpy="0 0 0"/>
+      <geometry>
+        <sphere radius="0.05"/>
+      </geometry>
+    </collision>
+  </link>
+  <gazebo reference="front_left_caster">
+    <material>Gazebo/Grey</material>
+    <mu1>0.0</mu1>
+    <mu2>0.0</mu2>
+  </gazebo>
+  <joint name="front_left_caster_joint" type="fixed">
+    <origin xyz="0.3 -0.7 -0.0926" rpy="0 0 0"/>
+    <parent link="chassibigga"/>
+    <child link="front_left_caster"/>
+  </joint>
+  <!-- Front Right Caster -->
+  <link name="front_right_caster">
+    <inertial>
+      <origin xyz="0 0 0" rpy="0 0 0"/>
+      <mass value="0.5"/>
+      <xacro:sphere_inertia m="0.5" r="0.05"/>
+    </inertial>
+    <visual>
+      <origin xyz="0 0 0" rpy="0 0 0"/>
+      <geometry>
+        <sphere radius="0.05"/>
+      </geometry>
+      <material name="caster_material">
+        <color rgba="0.5 0.5 0.5 1"/>
+      </material>
+    </visual>
+    <collision>
+      <origin xyz="0 0 0" rpy="0 0 0"/>
+      <geometry>
+        <sphere radius="0.05"/>
+      </geometry>
+    </collision>
+  </link>
+  <gazebo reference="front_right_caster">
+    <material>Gazebo/Grey</material>
+    <mu1>0.0</mu1>
+    <mu2>0.0</mu2>
+  </gazebo>
+  <joint name="front_right_caster_joint" type="fixed">
+    <origin xyz="-0.3 -0.7 -0.0926" rpy="0 0 0"/>
+    <parent link="chassibigga"/>
+    <child link="front_right_caster"/>
+  </joint>
+  <!-- ============================================ -->
+  <!-- CASTER WHEELS (Back - 2 wheels) -->
+  <!-- ============================================ -->
+  <!-- Back Left Caster -->
+  <link name="back_left_caster">
+    <inertial>
+      <origin xyz="0 0 0" rpy="0 0 0"/>
+      <mass value="0.5"/>
+      <xacro:sphere_inertia m="0.5" r="0.05"/>
+    </inertial>
+    <visual>
+      <origin xyz="0 0 0" rpy="0 0 0"/>
+      <geometry>
+        <sphere radius="0.05"/>
+      </geometry>
+      <material name="caster_material">
+        <color rgba="0.5 0.5 0.5 1"/>
+      </material>
+    </visual>
+    <collision>
+      <origin xyz="0 0 0" rpy="0 0 0"/>
+      <geometry>
+        <sphere radius="0.05"/>
+      </geometry>
+    </collision>
+  </link>
+  <gazebo reference="back_left_caster">
+    <material>Gazebo/Grey</material>
+    <mu1>0.0</mu1>
+    <mu2>0.0</mu2>
+  </gazebo>
+  <joint name="back_left_caster_joint" type="fixed">
+    <origin xyz="0.3 0.7 -0.0926" rpy="0 0 0"/>
+    <parent link="chassibigga"/>
+    <child link="back_left_caster"/>
+  </joint>
+  <!-- Back Right Caster -->
+  <link name="back_right_caster">
+    <inertial>
+      <origin xyz="0 0 0" rpy="0 0 0"/>
+      <mass value="0.5"/>
+      <xacro:sphere_inertia m="0.5" r="0.05"/>
+    </inertial>
+    <visual>
+      <origin xyz="0 0 0" rpy="0 0 0"/>
+      <geometry>
+        <sphere radius="0.05"/>
+      </geometry>
+      <material name="caster_material">
+        <color rgba="0.5 0.5 0.5 1"/>
+      </material>
+    </visual>
+    <collision>
+      <origin xyz="0 0 0" rpy="0 0 0"/>
+      <geometry>
+        <sphere radius="0.05"/>
+      </geometry>
+    </collision>
+  </link>
+  <gazebo reference="back_right_caster">
+    <material>Gazebo/Grey</material>
+    <mu1>0.0</mu1>
+    <mu2>0.0</mu2>
+  </gazebo>
+  <joint name="back_right_caster_joint" type="fixed">
+    <origin xyz="-0.3 0.7 -0.0926" rpy="0 0 0"/>
+    <parent link="chassibigga"/>
+    <child link="back_right_caster"/>
+  </joint>
+  <!-- ============================================ -->
+  <!-- DIFFERENTIAL DRIVE PLUGIN -->
+  <!-- ============================================ -->
+  <gazebo>
+    <plugin name="differential_drive_controller" filename="libgazebo_ros_diff_drive.so">
+      <ros>
+        <remapping>cmd_vel:=cmd_vel</remapping>
+        <remapping>odom:=odom</remapping>
+      </ros>
+      <update_rate>100.0</update_rate>
+      <left_joint>left_wheel_joint</left_joint>
+      <right_joint>right_wheel_joint</right_joint>
+      <wheel_separation>1.0</wheel_separation>
+      <wheel_diameter>0.2852</wheel_diameter>
+      <max_wheel_torque>200</max_wheel_torque>
+      <max_wheel_acceleration>10.0</max_wheel_acceleration>
+      <publish_odom>true</publish_odom>
+      <publish_odom_tf>true</publish_odom_tf>
+      <publish_wheel_tf>true</publish_wheel_tf>
+      <odometry_frame>odom</odometry_frame>
+      <robot_base_frame>base_link</robot_base_frame>
+    </plugin>
+  </gazebo>
+  <!-- ============================================ -->
+  <!-- TUGGER-TRAILER CONNECTION -->
+  <!-- ============================================ -->
+  <!-- Hitch point at the back of tugger (old base_link position) -->
+  <link name="hitch_link">
+    <inertial>
+      <origin xyz="0 0 0" rpy="0 0 0"/>
+      <mass value="1.0"/>
+      <inertia ixx="0.01" ixy="0" ixz="0" iyy="0.01" iyz="0" izz="0.01"/>
+    </inertial>
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
Commit message: :sparkles: fixed wheels visual orientation

File: urdf/glr.xacro (robot description, xacro)
@@ -78,5 +78,5 @@
     </inertial>
     <visual>
-      <origin xyz="0 0 0" rpy="1.5708 0 0"/>
+      <origin xyz="0 0 0" rpy="0 1.5708 0"/>
       <geometry>
         <cylinder radius="0.14260" length="0.08"/>
@@ -87,5 +87,5 @@
     </visual>
     <collision>
-      <origin xyz="0 0 0" rpy="1.5708 0 0"/>
+      <origin xyz="0 0 0" rpy="0 1.5708 0"/>
       <geometry>
         <cylinder radius="0.14260" length="0.08"/>
@@ -113,5 +113,5 @@
     </inertial>
     <visual>
-      <origin xyz="0 0 0" rpy="1.5708 0 0"/>
+      <origin xyz="0 0 0" rpy="0 1.5708 0"/>
       <geometry>
         <cylinder radius="0.14260" length="0.08"/>
@@ -122,5 +122,5 @@
     </visual>
     <collision>
-      <origin xyz="0 0 0" rpy="1.5708 0 0"/>
+      <origin xyz="0 0 0" rpy="0 1.5708 0"/>
       <geometry>
         <cylinder radius="0.14260" length="0.08"/>
