Commit message: :sparkles: added caster wheels joints

File: urdf/glr.xacro (robot description, xacro)
@@ -143,5 +143,20 @@
   <!-- CASTER WHEELS (Front - 2 wheels) -->
   <!-- ============================================ -->
-  <!-- Front Left Caster -->
+  <!-- Front Left Caster Mount -->
+  <link name="front_left_caster_mount">
+    <inertial>
+      <origin xyz="0 0 0" rpy="0 0 0"/>
+      <mass value="0.1"/>
+      <inertia ixx="0.0001" ixy="0" ixz="0" iyy="0.0001" iyz="0" izz="0.0001"/>
+    </inertial>
+  </link>
+  <joint name="front_left_caster_steering_joint" type="continuous">
+    <origin xyz="0.3 -0.7 -0.0926" rpy="0 0 0"/>
+    <parent link="chassibigga"/>
+    <child link="front_left_caster_mount"/>
+    <axis xyz="0 0 1"/>
+    <dynamics damping="0.0" friction="0.0"/>
+  </joint>
+  <!-- Front Left Caster Wheel -->
   <link name="front_left_caster">
     <inertial>
@@ -171,10 +186,27 @@
     <mu2>0.0</mu2>
   </gazebo>
-  <joint name="front_left_caster_joint" type="fixed">
-    <origin xyz="0.3 -0.7 -0.0926" rpy="0 0 0"/>
+  <joint name="front_left_caster_wheel_joint" type="continuous">
+    <origin xyz="0 0 0" rpy="0 0 0"/>
+    <parent link="front_left_caster_mount"/>
+    <child link="front_left_caster"/>
+    <axis xyz="1 0 0"/>
+    <dynamics damping="0.0" friction="0.0"/>
+  </joint>
+  <!-- Front Right Caster Mount -->
+  <link name="front_right_caster_mount">
+    <inertial>
+      <origin xyz="0 0 0" rpy="0 0 0"/>
+      <mass value="0.1"/>
+      <inertia ixx="0.0001" ixy="0" ixz="0" iyy="0.0001" iyz="0" izz="0.0001"/>
+    </inertial>
+  </link>
+  <joint name="front_right_caster_steering_joint" type="continuous">
+    <origin xyz="-0.3 -0.7 -0.0926" rpy="0 0 0"/>
     <parent link="chassibigga"/>
-    <child link="front_left_caster"/>
-  </joint>
-  <!-- Front Right Caster -->
+    <child link="front_right_caster_mount"/>
+    <axis xyz="0 0 1"/>
+    <dynamics damping="0.0" friction="0.0"/>
+  </joint>
+  <!-- Front Right Caster Wheel -->
   <link name="front_right_caster">
     <inertial>
@@ -204,13 +236,30 @@
     <mu2>0.0</mu2>
   </gazebo>
-  <joint name="front_right_caster_joint" type="fixed">
-    <origin xyz="-0.3 -0.7 -0.0926" rpy="0 0 0"/>
-    <parent link="chassibigga"/>
+  <joint name="front_right_caster_wheel_joint" type="continuous">
+    <origin xyz="0 0 0" rpy="0 0 0"/>
+    <parent link="front_right_caster_mount"/>
     <child link="front_right_caster"/>
+    <axis xyz="1 0 0"/>
+    <dynamics damping="0.0" friction="0.0"/>
   </joint>
   <!-- ============================================ -->
   <!-- CASTER WHEELS (Back - 2 wheels) -->
   <!-- ============================================ -->
-  <!-- Back Left Caster -->
+  <!-- Back Left Caster Mount -->
+  <link name="back_left_caster_mount">
+    <inertial>
+      <origin xyz="0 0 0" rpy="0 0 0"/>
+      <mass value="0.1"/>
+      <inertia ixx="0.0001" ixy="0" ixz="0" iyy="0.0001" iyz="0" izz="0.0001"/>
+    </inertial>
+  </link>
+  <joint name="back_left_caster_steering_joint" type="continuous">
+    <origin xyz="0.3 0.7 -0.0926" rpy="0 0 0"/>
+    <parent link="chassibigga"/>
+    <child link="back_left_caster_mount"/>
+    <axis xyz="0 0 1"/>
+    <dynamics damping="0.0" friction="0.0"/>
+  </joint>
+  <!-- Back Left Caster Wheel -->
   <link name="back_left_caster">
     <inertial>
@@ -240,10 +289,27 @@
     <mu2>0.0</mu2>
   </gazebo>
-  <joint name="back_left_caster_joint" type="fixed">
-    <origin xyz="0.3 0.7 -0.0926" rpy="0 0 0"/>
+  <joint name="back_left_caster_wheel_joint" type="continuous">
+    <origin xyz="0 0 0" rpy="0 0 0"/>
+    <parent link="back_left_caster_mount"/>
+    <child link="back_left_caster"/>
+    <axis xyz="1 0 0"/>
+    <dynamics damping="0.0" friction="0.0"/>
+  </joint>
+  <!-- Back Right Caster Mount -->
+  <link name="back_right_caster_mount">
+    <inertial>
+      <origin xyz="0 0 0" rpy="0 0 0"/>
+      <mass value="0.1"/>
+      <inertia ixx="0.0001" ixy="0" ixz="0" iyy="0.0001" iyz="0" izz="0.0001"/>
+    </inertial>
+  </link>
+  <joint name="back_right_caster_steering_joint" type="continuous">
+    <origin xyz="-0.3 0.7 -0.0926" rpy="0 0 0"/>
     <parent link="chassibigga"/>
-    <child link="back_left_caster"/>
-  </joint>
-  <!-- Back Right Caster -->
+    <child link="back_right_caster_mount"/>
+    <axis xyz="0 0 1"/>
+    <dynamics damping="0.0" friction="0.0"/>
+  </joint>
+  <!-- Back Right Caster Wheel -->
   <link name="back_right_caster">
     <inertial>
@@ -273,8 +339,10 @@
     <mu2>0.0</mu2>
   </gazebo>
-  <joint name="back_right_caster_joint" type="fixed">
-    <origin xyz="-0.3 0.7 -0.0926" rpy="0 0 0"/>
-    <parent link="chassibigga"/>
+  <joint name="back_right_caster_wheel_joint" type="continuous">
+    <origin xyz="0 0 0" rpy="0 0 0"/>
+    <parent link="back_right_caster_mount"/>
     <child link="back_right_caster"/>
+    <axis xyz="1 0 0"/>
+    <dynamics damping="0.0" friction="0.0"/>
   </joint>
   <!-- ============================================ -->
@@ -535,5 +603,5 @@
     <inertial>
       <origin
-        xyz="-0.08 0 0"
+        xyz="0 0 0"
         rpy="0 0 0" />
       <mass
@@ -543,8 +611,8 @@
     <visual>
       <origin
-        xyz="-0.08 0 0"
+        xyz="0 0 0"
         rpy="0 1.5708 0" />
       <geometry>
-        <cylinder radius="0.14260" length="0.16"/>
+        <cylinder radius="0.14260" length="0.08"/>
       </geometry>
       <material
@@ -556,8 +624,8 @@
     <collision>
       <origin
-        xyz="-0.08 0 0"
-        rpy="0 1.57 0" />
-      <geometry>
-        <sphere radius="0.14260"/>
+        xyz="0 0 0"
+        rpy="0 1.5708 0" />
+      <geometry>
+        <cylinder radius="0.14260" length="0.08"/>
       </geometry>
     </collision>
@@ -802,5 +870,5 @@
     <inertial>
       <origin
-        xyz="0.08 0 0"
+        xyz="0 0 0"
         rpy="0 0 0" />
       <mass
@@ -810,8 +878,8 @@
     <visual>
       <origin
-        xyz="0.08 0 0"
+        xyz="0 0 0"
         rpy="0 1.5708 0" />
       <geometry>
-        <cylinder radius="0.14260" length="0.16"/>
+        <cylinder radius="0.14260" length="0.08"/>
       </geometry>
       <material
@@ -823,8 +891,8 @@
     <collision>
       <origin
-        xyz="0.08 0 0"
+        xyz="0 0 0"
         rpy="0 1.5708 0" />
       <geometry>
-        <sphere radius="0.14260"/>
+        <cylinder radius="0.14260" length="0.08"/>
       </geometry>
     </collision>
@@ -925,5 +993,5 @@
     <inertial>
       <origin
-        xyz="-0.089466 6.8295E-06 -8.8605E-05"
+        xyz="0 0 0"
         rpy="0 0 0" />
       <mass
@@ -933,8 +1001,8 @@
     <visual>
       <origin
-        xyz="-0.08 0 0"
+        xyz="0 0 0"
         rpy="0 1.5708 0" />
       <geometry>
-        <cylinder radius="0.14260" length="0.16"/>
+        <cylinder radius="0.14260" length="0.08"/>
       </geometry>
       <material
@@ -946,8 +1014,8 @@
     <collision>
       <origin
-        xyz="-0.08 0 0"
-        rpy="0 1.57 0" />
-      <geometry>
-        <sphere radius="0.14260"/>
+        xyz="0 0 0"
+        rpy="0 1.5708 0" />
+      <geometry>
+        <cylinder radius="0.14260" length="0.08"/>
       </geometry>
     </collision>
@@ -1046,5 +1114,5 @@
     <inertial>
       <origin
-        xyz="0.08 0 0"
+        xyz="0 0 0"
         rpy="0 0 0" />
       <mass
@@ -1054,8 +1122,8 @@
     <visual>
       <origin
-        xyz="0.08 0 0"
+        xyz="0 0 0"
         rpy="0 1.5708 0" />
       <geometry>
-        <cylinder radius="0.14260" length="0.16"/>
+        <cylinder radius="0.14260" length="0.08"/>
       </geometry>
       <material
@@ -1067,8 +1135,8 @@
     <collision>
       <origin
-        xyz="0.08 0 0"
-        rpy="0 1.57 0" />
-      <geometry>
-        <sphere radius="0.14260"/>
+        xyz="0 0 0"
+        rpy="0 1.5708 0" />
+      <geometry>
+        <cylinder radius="0.14260" length="0.08"/>
       </geometry>
     </collision>

Commit message: :sparkles: changed tugger size

File: urdf/glr.xacro (robot description, xacro)
@@ -32,16 +32,16 @@
     <inertial>
       <origin
-        xyz="0 0 0.38"
+        xyz="0 0 0.155"
         rpy="0 0 0" />
       <mass
         value="555.02" />
-      <xacro:box_inertia m="555.02" w="0.9" d="1.6" h="1.1"/>
-    </inertial>
-    <visual>
-      <origin
-        xyz="0 0 0.38"
-        rpy="0 0 0" />
-      <geometry>
-          <box size="0.90 1.6 0.80"/>
+      <xacro:box_inertia m="555.02" w="0.5" d="0.7" h="0.31"/>
+    </inertial>
+    <visual>
+      <origin
+        xyz="0 0 0.155"
+        rpy="0 0 0" />
+      <geometry>
+          <box size="0.50 0.70 0.31"/>
       </geometry>
       <material
@@ -53,8 +53,8 @@
     <collision>
       <origin
-        xyz="0 0 0.38"
-        rpy="0 0 0" />
-      <geometry>
-          <box size="0.90 1.6 0.80"/>
+        xyz="0 0 0.155"
+        rpy="0 0 0" />
+      <geometry>
+          <box size="0.50 0.70 0.31"/>
       </geometry>
     </collision>
@@ -67,7 +67,4 @@
     <child link="chassibigga"/>
   </joint>
-  <!-- ============================================ -->
-  <!-- DIFFERENTIAL DRIVE WHEELS (Center - Traction) -->
-  <!-- ============================================ -->
   <!-- Left Traction Wheel -->
   <link name="left_wheel">
@@ -75,10 +72,10 @@
       <origin xyz="0 0 0" rpy="0 0 0"/>
       <mass value="12"/>
-      <xacro:sphere_inertia m="12" r="0.14260"/>
+      <xacro:sphere_inertia m="12" r="0.1"/>
     </inertial>
     <visual>
       <origin xyz="0 0 0" rpy="0 1.5708 0"/>
       <geometry>
-        <cylinder radius="0.14260" length="0.08"/>
+        <cylinder radius="0.1" length="0.08"/>
       </geometry>
       <material name="wheel_material">
@@ -89,5 +86,5 @@
       <origin xyz="0 0 0" rpy="0 1.5708 0"/>
       <geometry>
-        <cylinder radius="0.14260" length="0.08"/>
+        <cylinder radius="0.1" length="0.08"/>
       </geometry>
     </collision>
@@ -99,5 +96,5 @@
   </gazebo>
   <joint name="left_wheel_joint" type="continuous">
-    <origin xyz="0.5 0 0" rpy="0 0 0"/>
+    <origin xyz="0.25 0 0" rpy="0 0 0"/>
     <parent link="chassibigga"/>
     <child link="left_wheel"/>
@@ -110,10 +107,10 @@
       <origin xyz="0 0 0" rpy="0 0 0"/>
       <mass value="12"/>
-      <xacro:sphere_inertia m="12" r="0.14260"/>
+      <xacro:sphere_inertia m="12" r="0.1"/>
     </inertial>
     <visual>
       <origin xyz="0 0 0" rpy="0 1.5708 0"/>
       <geometry>
-        <cylinder radius="0.14260" length="0.08"/>
+        <cylinder radius="0.1" length="0.08"/>
       </geometry>
       <material name="wheel_material">
@@ -124,5 +121,5 @@
       <origin xyz="0 0 0" rpy="0 1.5708 0"/>
       <geometry>
-        <cylinder radius="0.14260" length="0.08"/>
+        <cylinder radius="0.1" length="0.08"/>
       </geometry>
     </collision>
@@ -134,5 +131,5 @@
   </gazebo>
   <joint name="right_wheel_joint" type="continuous">
-    <origin xyz="-0.5 0 0" rpy="0 0 0"/>
+    <origin xyz="-0.25 0 0" rpy="0 0 0"/>
     <parent link="chassibigga"/>
     <child link="right_wheel"/>
@@ -140,7 +137,4 @@
     <dynamics damping="0.1" friction="0.1"/>
   </joint>
-  <!-- ============================================ -->
-  <!-- CASTER WHEELS (Front - 2 wheels) -->
-  <!-- ============================================ -->
   <!-- Front Left Caster Mount -->
   <link name="front_left_caster_mount">
@@ -152,5 +146,5 @@
   </link>
   <joint name="front_left_caster_steering_joint" type="continuous">
-    <origin xyz="0.3 -0.7 -0.0926" rpy="0 0 0"/>
+    <origin xyz="0.2 -0.3 -0.0926" rpy="0 0 0"/>
     <parent link="chassibigga"/>
     <child link="front_left_caster_mount"/>
@@ -202,5 +196,5 @@
   </link>
   <joint name="front_right_caster_steering_joint" type="continuous">
-    <origin xyz="-0.3 -0.7 -0.0926" rpy="0 0 0"/>
+    <origin xyz="-0.2 -0.3 -0.0926" rpy="0 0 0"/>
     <parent link="chassibigga"/>
     <child link="front_right_caster_mount"/>
@@ -255,5 +249,5 @@
   </link>
   <joint name="back_left_caster_steering_joint" type="continuous">
-    <origin xyz="0.3 0.7 -0.0926" rpy="0 0 0"/>
+    <origin xyz="0.2 0.3 -0.0926" rpy="0 0 0"/>
     <parent link="chassibigga"/>
     <child link="back_left_caster_mount"/>
@@ -305,5 +299,5 @@
   </link>
   <joint name="back_right_caster_steering_joint" type="continuous">
-    <origin xyz="-0.3 0.7 -0.0926" rpy="0 0 0"/>
+    <origin xyz="-0.2 0.3 -0.0926" rpy="0 0 0"/>
     <parent link="chassibigga"/>
     <child link="back_right_caster_mount"/>
@@ -358,5 +352,5 @@
       <left_joint>left_wheel_joint</left_joint>
       <right_joint>right_wheel_joint</right_joint>
-      <wheel_separation>1.0</wheel_separation>
+      <wheel_separation>0.5</wheel_separation>
       <wheel_diameter>0.2852</wheel_diameter>
       <max_wheel_torque>200</max_wheel_torque>
@@ -399,5 +393,5 @@
   </gazebo>
   <joint name="hitch_joint" type="fixed">
-    <origin xyz="0 0.8 0.14260" rpy="0 0 0"/>
+    <origin xyz="0 0.35 0.14260" rpy="0 0 0"/>
     <parent link="chassibigga"/>
     <child link="hitch_link"/>
@@ -728,13 +722,4 @@
       k_velocity="0" />
   </joint>
-  <!-- <transmission name="transmission_common">
-    <type>transmission_interface/SimpleTransmission</type>
-    <joint name="eixorodavolantebigga_steer">
-      <hardwareInterface>hardware_interface/PositionJointInterface</hardwareInterface>
-    </joint>
-    <joint name="eixorodeirodiant2">
-      <hardwareInterface>hardware_interface/PositionJointInterface</hardwareInterface>
-    </joint>
-  </transmission> -->
   <gazebo>
     <joint name='barradiant1_JOINT_1' type='revolute'>
@@ -1194,5 +1179,5 @@
     <parent link="chassibigga"/>
     <child link="lidar_link"/>
-    <origin xyz="0 -0.8 0.82" rpy="0 0 0"/>
+    <origin xyz="0 -0.25 0.37" rpy="0 0 0"/>
   </joint>
   <gazebo reference="lidar_link">

Commit message: :sparkles: fixed wheels position

File: urdf/glr.xacro (robot description, xacro)
@@ -1,4 +1,8 @@
 <?xml version="1.0" encoding="utf-8"?>
 <robot name="glr_description" xmlns:xacro="http://ros.org/wiki/xacro">
+  <!-- Wheel properties -->
+  <xacro:property name="wheel_radius" value="0.1" />
+  <xacro:property name="wheel_width" value="0.08" />
+  <xacro:property name="caster_radius" value="0.05" />
   <!-- Define intertial property macros  -->
   <xacro:macro name="box_inertia" params="m w d h">
@@ -66,4 +70,5 @@
     <parent link="base_link"/>
     <child link="chassibigga"/>
+    <origin xyz="0 0 ${wheel_radius}" rpy="0 0 0"/>
   </joint>
   <!-- Left Traction Wheel -->
@@ -72,10 +77,10 @@
       <origin xyz="0 0 0" rpy="0 0 0"/>
       <mass value="12"/>
-      <xacro:sphere_inertia m="12" r="0.1"/>
+      <xacro:sphere_inertia m="12" r="${wheel_radius}"/>
     </inertial>
     <visual>
       <origin xyz="0 0 0" rpy="0 1.5708 0"/>
       <geometry>
-        <cylinder radius="0.1" length="0.08"/>
+        <cylinder radius="${wheel_radius}" length="${wheel_width}"/>
       </geometry>
       <material name="wheel_material">
@@ -86,5 +91,5 @@
       <origin xyz="0 0 0" rpy="0 1.5708 0"/>
       <geometry>
-        <cylinder radius="0.1" length="0.08"/>
+        <cylinder radius="${wheel_radius}" length="${wheel_width}"/>
       </geometry>
     </collision>
@@ -107,10 +112,10 @@
       <origin xyz="0 0 0" rpy="0 0 0"/>
       <mass value="12"/>
-      <xacro:sphere_inertia m="12" r="0.1"/>
+      <xacro:sphere_inertia m="12" r="${wheel_radius}"/>
     </inertial>
     <visual>
       <origin xyz="0 0 0" rpy="0 1.5708 0"/>
       <geometry>
-        <cylinder radius="0.1" length="0.08"/>
+        <cylinder radius="${wheel_radius}" length="${wheel_width}"/>
       </geometry>
       <material name="wheel_material">
@@ -121,5 +126,5 @@
       <origin xyz="0 0 0" rpy="0 1.5708 0"/>
       <geometry>
-        <cylinder radius="0.1" length="0.08"/>
+        <cylinder radius="${wheel_radius}" length="${wheel_width}"/>
       </geometry>
     </collision>
@@ -146,5 +151,5 @@
   </link>
   <joint name="front_left_caster_steering_joint" type="continuous">
-    <origin xyz="0.2 -0.3 -0.0926" rpy="0 0 0"/>
+    <origin xyz="0.2 -0.3 ${-wheel_radius + caster_radius}" rpy="0 0 0"/>
     <parent link="chassibigga"/>
     <child link="front_left_caster_mount"/>
@@ -157,10 +162,10 @@
       <origin xyz="0 0 0" rpy="0 0 0"/>
       <mass value="0.5"/>
-      <xacro:sphere_inertia m="0.5" r="0.05"/>
-    </inertial>
-    <visual>
-      <origin xyz="0 0 0" rpy="0 0 0"/>
-      <geometry>
-        <sphere radius="0.05"/>
+      <xacro:sphere_inertia m="0.5" r="${caster_radius}"/>
+    </inertial>
+    <visual>
+      <origin xyz="0 0 0" rpy="0 0 0"/>
+      <geometry>
+        <sphere radius="${caster_radius}"/>
       </geometry>
       <material name="caster_material">
@@ -171,5 +176,5 @@
       <origin xyz="0 0 0" rpy="0 0 0"/>
       <geometry>
-        <sphere radius="0.05"/>
+        <sphere radius="${caster_radius}"/>
       </geometry>
     </collision>
@@ -196,5 +201,5 @@
   </link>
   <joint name="front_right_caster_steering_joint" type="continuous">
-    <origin xyz="-0.2 -0.3 -0.0926" rpy="0 0 0"/>
+    <origin xyz="-0.2 -0.3 ${-wheel_radius + caster_radius}" rpy="0 0 0"/>
     <parent link="chassibigga"/>
     <child link="front_right_caster_mount"/>
@@ -207,10 +212,10 @@
       <origin xyz="0 0 0" rpy="0 0 0"/>
       <mass value="0.5"/>
-      <xacro:sphere_inertia m="0.5" r="0.05"/>
-    </inertial>
-    <visual>
-      <origin xyz="0 0 0" rpy="0 0 0"/>
-      <geometry>
-        <sphere radius="0.05"/>
+      <xacro:sphere_inertia m="0.5" r="${caster_radius}"/>
+    </inertial>
+    <visual>
+      <origin xyz="0 0 0" rpy="0 0 0"/>
+      <geometry>
+        <sphere radius="${caster_radius}"/>
       </geometry>
       <material name="caster_material">
@@ -221,5 +226,5 @@
       <origin xyz="0 0 0" rpy="0 0 0"/>
       <geometry>
-        <sphere radius="0.05"/>
+        <sphere radius="${caster_radius}"/>
       </geometry>
     </collision>
@@ -249,5 +254,5 @@
   </link>
   <joint name="back_left_caster_steering_joint" type="continuous">
-    <origin xyz="0.2 0.3 -0.0926" rpy="0 0 0"/>
+    <origin xyz="0.2 0.3 ${-wheel_radius + caster_radius}" rpy="0 0 0"/>
     <parent link="chassibigga"/>
     <child link="back_left_caster_mount"/>
@@ -260,10 +265,10 @@
       <origin xyz="0 0 0" rpy="0 0 0"/>
       <mass value="0.5"/>
-      <xacro:sphere_inertia m="0.5" r="0.05"/>
-    </inertial>
-    <visual>
-      <origin xyz="0 0 0" rpy="0 0 0"/>
-      <geometry>
-        <sphere radius="0.05"/>
+      <xacro:sphere_inertia m="0.5" r="${caster_radius}"/>
+    </inertial>
+    <visual>
+      <origin xyz="0 0 0" rpy="0 0 0"/>
+      <geometry>
+        <sphere radius="${caster_radius}"/>
       </geometry>
       <material name="caster_material">
@@ -274,5 +279,5 @@
       <origin xyz="0 0 0" rpy="0 0 0"/>
       <geometry>
-        <sphere radius="0.05"/>
+        <sphere radius="${caster_radius}"/>
       </geometry>
     </collision>
@@ -299,5 +304,5 @@
   </link>
   <joint name="back_right_caster_steering_joint" type="continuous">
-    <origin xyz="-0.2 0.3 -0.0926" rpy="0 0 0"/>
+    <origin xyz="-0.2 0.3 ${-wheel_radius + caster_radius}" rpy="0 0 0"/>
     <parent link="chassibigga"/>
     <child link="back_right_caster_mount"/>
@@ -310,10 +315,10 @@
       <origin xyz="0 0 0" rpy="0 0 0"/>
       <mass value="0.5"/>
-      <xacro:sphere_inertia m="0.5" r="0.05"/>
-    </inertial>
-    <visual>
-      <origin xyz="0 0 0" rpy="0 0 0"/>
-      <geometry>
-        <sphere radius="0.05"/>
+      <xacro:sphere_inertia m="0.5" r="${caster_radius}"/>
+    </inertial>
+    <visual>
+      <origin xyz="0 0 0" rpy="0 0 0"/>
+      <geometry>
+        <sphere radius="${caster_radius}"/>
       </geometry>
       <material name="caster_material">
@@ -324,5 +329,5 @@
       <origin xyz="0 0 0" rpy="0 0 0"/>
       <geometry>
-        <sphere radius="0.05"/>
+        <sphere radius="${caster_radius}"/>
       </geometry>
     </collision>
@@ -353,5 +358,5 @@
       <right_joint>right_wheel_joint</right_joint>
       <wheel_separation>0.5</wheel_separation>
-      <wheel_diameter>0.2852</wheel_diameter>
+      <wheel_diameter>${2 * wheel_radius}</wheel_diameter>
       <max_wheel_torque>200</max_wheel_torque>
       <max_wheel_acceleration>10.0</max_wheel_acceleration>
@@ -1179,5 +1184,5 @@
     <parent link="chassibigga"/>
     <child link="lidar_link"/>
-    <origin xyz="0 -0.25 0.37" rpy="0 0 0"/>
+    <origin xyz="0 -0.25 0.155" rpy="0 0 0"/>
   </joint>
   <gazebo reference="lidar_link">
