Commit message: :sparkles: added trailer wheels variables

File: urdf/glr.xacro (robot description, xacro)
@@ -4,5 +4,7 @@
   <xacro:property name="wheel_radius" value="0.1" />
   <xacro:property name="wheel_width" value="0.08" />
-  <xacro:property name="caster_radius" value="0.05" />
+  <xacro:property name="caster_radius" value="0.08" />
+  <xacro:property name="trailer_wheel_radius" value="0.1" />
+  <xacro:property name="trailer_wheel_width" value="0.08" />
   <!-- Define intertial property macros  -->
   <xacro:macro name="box_inertia" params="m w d h">
@@ -142,5 +144,8 @@
     <dynamics damping="0.1" friction="0.1"/>
   </joint>
-  <!-- Front Left Caster Mount -->
+  <!-- ============================================ -->
+  <!-- CASTER WHEELS COMMENTED FOR TESTING -->
+  <!-- ============================================ -->
+  <!--
   <link name="front_left_caster_mount">
     <inertial>
@@ -157,5 +162,4 @@
     <dynamics damping="0.0" friction="0.0"/>
   </joint>
-  <!-- Front Left Caster Wheel -->
   <link name="front_left_caster">
     <inertial>
@@ -192,5 +196,4 @@
     <dynamics damping="0.0" friction="0.0"/>
   </joint>
-  <!-- Front Right Caster Mount -->
   <link name="front_right_caster_mount">
     <inertial>
@@ -207,5 +210,4 @@
     <dynamics damping="0.0" friction="0.0"/>
   </joint>
-  <!-- Front Right Caster Wheel -->
   <link name="front_right_caster">
     <inertial>
@@ -242,8 +244,4 @@
     <dynamics damping="0.0" friction="0.0"/>
   </joint>
-  <!-- ============================================ -->
-  <!-- CASTER WHEELS (Back - 2 wheels) -->
-  <!-- ============================================ -->
-  <!-- Back Left Caster Mount -->
   <link name="back_left_caster_mount">
     <inertial>
@@ -260,5 +258,4 @@
     <dynamics damping="0.0" friction="0.0"/>
   </joint>
-  <!-- Back Left Caster Wheel -->
   <link name="back_left_caster">
     <inertial>
@@ -295,5 +292,4 @@
     <dynamics damping="0.0" friction="0.0"/>
   </joint>
-  <!-- Back Right Caster Mount -->
   <link name="back_right_caster_mount">
     <inertial>
@@ -310,5 +306,4 @@
     <dynamics damping="0.0" friction="0.0"/>
   </joint>
-  <!-- Back Right Caster Wheel -->
   <link name="back_right_caster">
     <inertial>
@@ -345,4 +340,5 @@
     <dynamics damping="0.0" friction="0.0"/>
   </joint>
+  -->
   <!-- ============================================ -->
   <!-- DIFFERENTIAL DRIVE PLUGIN -->
@@ -606,5 +602,5 @@
       <mass
         value="2" />
-      <xacro:sphere_inertia m="2" r="0.14260"/>
+      <xacro:sphere_inertia m="2" r="${trailer_wheel_radius}"/>
     </inertial>
     <visual>
@@ -613,5 +609,5 @@
         rpy="0 1.5708 0" />
       <geometry>
-        <cylinder radius="0.14260" length="0.08"/>
+        <cylinder radius="${trailer_wheel_radius}" length="${trailer_wheel_width}"/>
       </geometry>
       <material
@@ -626,5 +622,5 @@
         rpy="0 1.5708 0" />
       <geometry>
-        <cylinder radius="0.14260" length="0.08"/>
+        <cylinder radius="${trailer_wheel_radius}" length="${trailer_wheel_width}"/>
       </geometry>
     </collision>
@@ -864,5 +860,5 @@
       <mass
         value="2" />
-      <xacro:sphere_inertia m="2" r="0.14260"/>
+      <xacro:sphere_inertia m="2" r="${trailer_wheel_radius}"/>
     </inertial>
     <visual>
@@ -871,5 +867,5 @@
         rpy="0 1.5708 0" />
       <geometry>
-        <cylinder radius="0.14260" length="0.08"/>
+        <cylinder radius="${trailer_wheel_radius}" length="${trailer_wheel_width}"/>
       </geometry>
       <material
@@ -884,5 +880,5 @@
         rpy="0 1.5708 0" />
       <geometry>
-        <cylinder radius="0.14260" length="0.08"/>
+        <cylinder radius="${trailer_wheel_radius}" length="${trailer_wheel_width}"/>
       </geometry>
     </collision>
@@ -987,5 +983,5 @@
       <mass
         value="2" />
-      <xacro:sphere_inertia m="2" r="0.14260"/>
+      <xacro:sphere_inertia m="2" r="${trailer_wheel_radius}"/>
     </inertial>
     <visual>
@@ -994,5 +990,5 @@
         rpy="0 1.5708 0" />
       <geometry>
-        <cylinder radius="0.14260" length="0.08"/>
+        <cylinder radius="${trailer_wheel_radius}" length="${trailer_wheel_width}"/>
       </geometry>
       <material
@@ -1007,5 +1003,5 @@
         rpy="0 1.5708 0" />
       <geometry>
-        <cylinder radius="0.14260" length="0.08"/>
+        <cylinder radius="${trailer_wheel_radius}" length="${trailer_wheel_width}"/>
       </geometry>
     </collision>
@@ -1108,5 +1104,5 @@
       <mass
         value="2" />
-      <xacro:sphere_inertia m="2" r="0.14260"/>
+      <xacro:sphere_inertia m="2" r="${trailer_wheel_radius}"/>
     </inertial>
     <visual>
@@ -1115,5 +1111,5 @@
         rpy="0 1.5708 0" />
       <geometry>
-        <cylinder radius="0.14260" length="0.08"/>
+        <cylinder radius="${trailer_wheel_radius}" length="${trailer_wheel_width}"/>
       </geometry>
       <material
@@ -1128,5 +1124,5 @@
         rpy="0 1.5708 0" />
       <geometry>
-        <cylinder radius="0.14260" length="0.08"/>
+        <cylinder radius="${trailer_wheel_radius}" length="${trailer_wheel_width}"/>
       </geometry>
     </collision>
@@ -1184,5 +1180,5 @@
     <parent link="chassibigga"/>
     <child link="lidar_link"/>
-    <origin xyz="0 -0.25 0.155" rpy="0 0 0"/>
+    <origin xyz="0 -0.25 0.34" rpy="0 0 0"/>
   </joint>
   <gazebo reference="lidar_link">
@@ -1190,5 +1186,5 @@
     <sensor type="ray" name="lidar_sensor">
       <pose>0 0 0 0 0 0</pose>
-      <visualize>true</visualize>
+      <visualize>false</visualize>
       <update_rate>10</update_rate>
       <ray>

Commit message: :fire: removed gazebo configs

File: urdf/glr.xacro (robot description, xacro)
@@ -1,1220 +1,7 @@
 <?xml version="1.0" encoding="utf-8"?>
 <robot name="glr_description" xmlns:xacro="http://ros.org/wiki/xacro">
-  <!-- Wheel properties -->
-  <xacro:property name="wheel_radius" value="0.1" />
-  <xacro:property name="wheel_width" value="0.08" />
-  <xacro:property name="caster_radius" value="0.08" />
-  <xacro:property name="trailer_wheel_radius" value="0.1" />
-  <xacro:property name="trailer_wheel_width" value="0.08" />
-  <!-- Define intertial property macros  -->
-  <xacro:macro name="box_inertia" params="m w d h">
-    <inertia ixx="${1*(m/12) * (h*h + d*d)}" ixy="0.0" ixz="0.0" iyy="${1*(m/12) * (w*w + d*d)}" iyz="0.0" izz="${1*(m/12) * (w*w + h*h)}"/>
-  </xacro:macro>
-  <xacro:macro name="sphere_inertia" params="m r">
-    <inertia ixx="${1*(2/5) * m * (r*r)}" ixy="0.0" ixz="0.0" iyy="${1*(2/5) * m * (r*r)}" iyz="0.0" izz="${1*(2/5) * m * (r*r)}"/>
-  </xacro:macro>
-  <xacro:macro name="cylinder_inertia" params="m r h">
-    <inertial>
-      <!-- <origin xyz="0 0 0" rpy="${pi/2} 0 0" /> -->
-      <mass value="${m}"/>
-      <inertia  ixx="${m*(3*r*r+h*h)/12}" ixy = "0" ixz = "0" iyy="${m*(3*r*r+h*h)/12}" iyz = "0" izz="${m*r*r/2}" />
-      <!-- <inertia ixx="${(m/12) * (3*r*r + h*h)}" ixy = "0" ixz = "0" iyy="${(m/12) * (3*r*r + h*h)}" iyz = "0" izz="${(m/2) * (r*r)}"/> -->
-    </inertial>
-  </xacro:macro>
-  <!--Robot description  -->
-  <link name="base_link"/>
-  <!-- Robot Footprint -->
-  <link name="base_footprint"/>
-  <joint name="base_joint" type="fixed">
-    <parent link="base_link"/>
-    <child link="base_footprint"/>
-    <origin xyz="0 0 0" rpy="0 0 0"/>
-  </joint>
-  <!-- Tugger -->
-  <link name="chassibigga">
-    <origin
-        xyz="0 0 0"
-        rpy="0 0 0" />
-    <inertial>
-      <origin
-        xyz="0 0 0.155"
-        rpy="0 0 0" />
-      <mass
-        value="555.02" />
-      <xacro:box_inertia m="555.02" w="0.5" d="0.7" h="0.31"/>
-    </inertial>
-    <visual>
-      <origin
-        xyz="0 0 0.155"
-        rpy="0 0 0" />
-      <geometry>
-          <box size="0.50 0.70 0.31"/>
-      </geometry>
-      <material
-        name="">
-        <color
-          rgba="0.64706 0.61961 0.58824 1" />
-      </material>
-    </visual>
-    <collision>
-      <origin
-        xyz="0 0 0.155"
-        rpy="0 0 0" />
-      <geometry>
-          <box size="0.50 0.70 0.31"/>
-      </geometry>
-    </collision>
-  </link>
-  <gazebo reference="chassibigga">
-    <material>Gazebo/Orange</material>
-  </gazebo>
-  <joint name="base_chassi_joint" type="fixed">
-    <parent link="base_link"/>
-    <child link="chassibigga"/>
-    <origin xyz="0 0 ${wheel_radius}" rpy="0 0 0"/>
-  </joint>
-  <!-- Left Traction Wheel -->
-  <link name="left_wheel">
-    <inertial>
-      <origin xyz="0 0 0" rpy="0 0 0"/>
-      <mass value="12"/>
-      <xacro:sphere_inertia m="12" r="${wheel_radius}"/>
-    </inertial>
-    <visual>
-      <origin xyz="0 0 0" rpy="0 1.5708 0"/>
-      <geometry>
-        <cylinder radius="${wheel_radius}" length="${wheel_width}"/>
-      </geometry>
-      <material name="wheel_material">
-        <color rgba="0.29804 0.29804 0.29804 1"/>
-      </material>
-    </visual>
-    <collision>
-      <origin xyz="0 0 0" rpy="0 1.5708 0"/>
-      <geometry>
-        <cylinder radius="${wheel_radius}" length="${wheel_width}"/>
-      </geometry>
-    </collision>
-  </link>
-  <gazebo reference="left_wheel">
-    <material>Gazebo/Black</material>
-    <mu1>1.0</mu1>
-    <mu2>1.0</mu2>
-  </gazebo>
-  <joint name="left_wheel_joint" type="continuous">
-    <origin xyz="0.25 0 0" rpy="0 0 0"/>
-    <parent link="chassibigga"/>
-    <child link="left_wheel"/>
-    <axis xyz="1 0 0"/>
-    <dynamics damping="0.1" friction="0.1"/>
-  </joint>
-  <!-- Right Traction Wheel -->
-  <link name="right_wheel">
-    <inertial>
-      <origin xyz="0 0 0" rpy="0 0 0"/>
-      <mass value="12"/>
-      <xacro:sphere_inertia m="12" r="${wheel_radius}"/>
-    </inertial>
-    <visual>
-      <origin xyz="0 0 0" rpy="0 1.5708 0"/>
-      <geometry>
-        <cylinder radius="${wheel_radius}" length="${wheel_width}"/>
-      </geometry>
-      <material name="wheel_material">
-        <color rgba="0.29804 0.29804 0.29804 1"/>
-      </material>
-    </visual>
-    <collision>
-      <origin xyz="0 0 0" rpy="0 1.5708 0"/>
-      <geometry>
-        <cylinder radius="${wheel_radius}" length="${wheel_width}"/>
-      </geometry>
-    </collision>
-  </link>
-  <gazebo reference="right_wheel">
-    <material>Gazebo/Black</material>
-    <mu1>1.0</mu1>
-    <mu2>1.0</mu2>
-  </gazebo>
-  <joint name="right_wheel_joint" type="continuous">
-    <origin xyz="-0.25 0 0" rpy="0 0 0"/>
-    <parent link="chassibigga"/>
-    <child link="right_wheel"/>
-    <axis xyz="1 0 0"/>
-    <dynamics damping="0.1" friction="0.1"/>
-  </joint>
-  <!-- ============================================ -->
-  <!-- CASTER WHEELS COMMENTED FOR TESTING -->
-  <!-- ============================================ -->
-  <!--
-  <link name="front_left_caster_mount">
-    <inertial>
-      <origin xyz="0 0 0" rpy="0 0 0"/>
-      <mass value="0.1"/>
-      <inertia ixx="0.0001" ixy="0" ixz="0" iyy="0.0001" iyz="0" izz="0.0001"/>
-    </inertial>
-  </link>
-  <joint name="front_left_caster_steering_joint" type="continuous">
-    <origin xyz="0.2 -0.3 ${-wheel_radius + caster_radius}" rpy="0 0 0"/>
-    <parent link="chassibigga"/>
-    <child link="front_left_caster_mount"/>
-    <axis xyz="0 0 1"/>
-    <dynamics damping="0.0" friction="0.0"/>
-  </joint>
-  <link name="front_left_caster">
-    <inertial>
-      <origin xyz="0 0 0" rpy="0 0 0"/>
-      <mass value="0.5"/>
-      <xacro:sphere_inertia m="0.5" r="${caster_radius}"/>
-    </inertial>
-    <visual>
-      <origin xyz="0 0 0" rpy="0 0 0"/>
-      <geometry>
-        <sphere radius="${caster_radius}"/>
-      </geometry>
-      <material name="caster_material">
-        <color rgba="0.5 0.5 0.5 1"/>
-      </material>
-    </visual>
-    <collision>
-      <origin xyz="0 0 0" rpy="0 0 0"/>
-      <geometry>
-        <sphere radius="${caster_radius}"/>
-      </geometry>
-    </collision>
-  </link>
-  <gazebo reference="front_left_caster">
-    <material>Gazebo/Grey</material>
-    <mu1>0.0</mu1>
-    <mu2>0.0</mu2>
-  </gazebo>
-  <joint name="front_left_caster_wheel_joint" type="continuous">
-    <origin xyz="0 0 0" rpy="0 0 0"/>
-    <parent link="front_left_caster_mount"/>
-    <child link="front_left_caster"/>
-    <axis xyz="1 0 0"/>
-    <dynamics damping="0.0" friction="0.0"/>
-  </joint>
-  <link name="front_right_caster_mount">
-    <inertial>
-      <origin xyz="0 0 0" rpy="0 0 0"/>
-      <mass value="0.1"/>
-      <inertia ixx="0.0001" ixy="0" ixz="0" iyy="0.0001" iyz="0" izz="0.0001"/>
-    </inertial>
-  </link>
-  <joint name="front_right_caster_steering_joint" type="continuous">
-    <origin xyz="-0.2 -0.3 ${-wheel_radius + caster_radius}" rpy="0 0 0"/>
-    <parent link="chassibigga"/>
-    <child link="front_right_caster_mount"/>
-    <axis xyz="0 0 1"/>
-    <dynamics damping="0.0" friction="0.0"/>
-  </joint>
-  <link name="front_right_caster">
-    <inertial>
-      <origin xyz="0 0 0" rpy="0 0 0"/>
-      <mass value="0.5"/>
-      <xacro:sphere_inertia m="0.5" r="${caster_radius}"/>
-    </inertial>
-    <visual>
-      <origin xyz="0 0 0" rpy="0 0 0"/>
-      <geometry>
-        <sphere radius="${caster_radius}"/>
-      </geometry>
-      <material name="caster_material">
-        <color rgba="0.5 0.5 0.5 1"/>
-      </material>
-    </visual>
-    <collision>
-      <origin xyz="0 0 0" rpy="0 0 0"/>
-      <geometry>
-        <sphere radius="${caster_radius}"/>
-      </geometry>
-    </collision>
-  </link>
-  <gazebo reference="front_right_caster">
-    <material>Gazebo/Grey</material>
-    <mu1>0.0</mu1>
-    <mu2>0.0</mu2>
-  </gazebo>
-  <joint name="front_right_caster_wheel_joint" type="continuous">
-    <origin xyz="0 0 0" rpy="0 0 0"/>
-    <parent link="front_right_caster_mount"/>
-    <child link="front_right_caster"/>
-    <axis xyz="1 0 0"/>
-    <dynamics damping="0.0" friction="0.0"/>
-  </joint>
-  <link name="back_left_caster_mount">
-    <inertial>
-      <origin xyz="0 0 0" rpy="0 0 0"/>
-      <mass value="0.1"/>
-      <inertia ixx="0.0001" ixy="0" ixz="0" iyy="0.0001" iyz="0" izz="0.0001"/>
-    </inertial>
-  </link>
-  <joint name="back_left_caster_steering_joint" type="continuous">
-    <origin xyz="0.2 0.3 ${-wheel_radius + caster_radius}" rpy="0 0 0"/>
-    <parent link="chassibigga"/>
-    <child link="back_left_caster_mount"/>
-    <axis xyz="0 0 1"/>
-    <dynamics damping="0.0" friction="0.0"/>
-  </joint>
-  <link name="back_left_caster">
-    <inertial>
-      <origin xyz="0 0 0" rpy="0 0 0"/>
-      <mass value="0.5"/>
-      <xacro:sphere_inertia m="0.5" r="${caster_radius}"/>
-    </inertial>
-    <visual>
-      <origin xyz="0 0 0" rpy="0 0 0"/>
-      <geometry>
-        <sphere radius="${caster_radius}"/>
-      </geometry>
-      <material name="caster_material">
-        <color rgba="0.5 0.5 0.5 1"/>
-      </material>
-    </visual>
-    <collision>
-      <origin xyz="0 0 0" rpy="0 0 0"/>
-      <geometry>
-        <sphere radius="${caster_radius}"/>
-      </geometry>
-    </collision>
-  </link>
-  <gazebo reference="back_left_caster">
-    <material>Gazebo/Grey</material>
-    <mu1>0.0</mu1>
-    <mu2>0.0</mu2>
-  </gazebo>
-  <joint name="back_left_caster_wheel_joint" type="continuous">
-    <origin xyz="0 0 0" rpy="0 0 0"/>
-    <parent link="back_left_caster_mount"/>
-    <child link="back_left_caster"/>
-    <axis xyz="1 0 0"/>
-    <dynamics damping="0.0" friction="0.0"/>
-  </joint>
-  <link name="back_right_caster_mount">
-    <inertial>
-      <origin xyz="0 0 0" rpy="0 0 0"/>
-      <mass value="0.1"/>
-      <inertia ixx="0.0001" ixy="0" ixz="0" iyy="0.0001" iyz="0" izz="0.0001"/>
-    </inertial>
-  </link>
-  <joint name="back_right_caster_steering_joint" type="continuous">
-    <origin xyz="-0.2 0.3 ${-wheel_radius + caster_radius}" rpy="0 0 0"/>
-    <parent link="chassibigga"/>
-    <child link="back_right_caster_mount"/>
-    <axis xyz="0 0 1"/>
-    <dynamics damping="0.0" friction="0.0"/>
-  </joint>
-  <link name="back_right_caster">
-    <inertial>
-      <origin xyz="0 0 0" rpy="0 0 0"/>
-      <mass value="0.5"/>
-      <xacro:sphere_inertia m="0.5" r="${caster_radius}"/>
-    </inertial>
-    <visual>
-      <origin xyz="0 0 0" rpy="0 0 0"/>
-      <geometry>
-        <sphere radius="${caster_radius}"/>
-      </geometry>
-      <material name="caster_material">
-        <color rgba="0.5 0.5 0.5 1"/>
-      </material>
-    </visual>
-    <collision>
-      <origin xyz="0 0 0" rpy="0 0 0"/>
-      <geometry>
-        <sphere radius="${caster_radius}"/>
-      </geometry>
-    </collision>
-  </link>
-  <gazebo reference="back_right_caster">
-    <material>Gazebo/Grey</material>
-    <mu1>0.0</mu1>
-    <mu2>0.0</mu2>
-  </gazebo>
-  <joint name="back_right_caster_wheel_joint" type="continuous">
-    <origin xyz="0 0 0" rpy="0 0 0"/>
-    <parent link="back_right_caster_mount"/>
-    <child link="back_right_caster"/>
-    <axis xyz="1 0 0"/>
-    <dynamics damping="0.0" friction="0.0"/>
-  </joint>
-  -->
-  <!-- ============================================ -->
-  <!-- DIFFERENTIAL DRIVE PLUGIN -->
-  <!-- ============================================ -->
-  <gazebo>
-    <plugin name="differential_drive_controller" filename="libgazebo_ros_diff_drive.so">
-      <ros>
-        <remapping>cmd_vel:=cmd_vel</remapping>
-        <remapping>odom:=odom</remapping>
-      </ros>
-      <update_rate>100.0</update_rate>
-      <left_joint>left_wheel_joint</left_joint>
-      <right_joint>right_wheel_joint</right_joint>
-      <wheel_separation>0.5</wheel_separation>
-      <wheel_diameter>${2 * wheel_radius}</wheel_diameter>
-      <max_wheel_torque>200</max_wheel_torque>
-      <max_wheel_acceleration>10.0</max_wheel_acceleration>
-      <publish_odom>true</publish_odom>
-      <publish_odom_tf>true</publish_odom_tf>
-      <publish_wheel_tf>true</publish_wheel_tf>
-      <odometry_frame>odom</odometry_frame>
-      <robot_base_frame>base_link</robot_base_frame>
-    </plugin>
-  </gazebo>
-  <!-- ============================================ -->
-  <!-- TUGGER-TRAILER CONNECTION -->
-  <!-- ============================================ -->
-  <!-- Hitch point at the back of tugger (old base_link position) -->
-  <link name="hitch_link">
-    <inertial>
-      <origin xyz="0 0 0" rpy="0 0 0"/>
-      <mass value="1.0"/>
-      <inertia ixx="0.01" ixy="0" ixz="0" iyy="0.01" iyz="0" izz="0.01"/>
-    </inertial>
-    <visual>
-      <origin xyz="0 0 0" rpy="0 0 0"/>
-      <geometry>
-        <cylinder radius="0.05" length="0.1"/>
-      </geometry>
-      <material name="hitch_material">
-        <color rgba="0.3 0.3 0.3 1"/>
-      </material>
-    </visual>
-    <collision>
-      <origin xyz="0 0 0" rpy="0 0 0"/>
-      <geometry>
-        <cylinder radius="0.05" length="0.1"/>
-      </geometry>
-    </collision>
-  </link>
-  <gazebo reference="hitch_link">
-    <material>Gazebo/DarkGrey</material>
-  </gazebo>
-  <joint name="hitch_joint" type="fixed">
-    <origin xyz="0 0.35 0.14260" rpy="0 0 0"/>
-    <parent link="chassibigga"/>
-    <child link="hitch_link"/>
-  </joint>
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