Commit message: :sparkles: xacros segmentation

File: urdf/glr.xacro (robot description, xacro)
@@ -1,7 +1,19 @@
 <?xml version="1.0" encoding="utf-8"?>
 <robot name="glr_description" xmlns:xacro="http://ros.org/wiki/xacro">
-  <!-- Include URDF definitions -->
-  <xacro:include filename="$(find glr_description)/urdf/glr_urdf.xacro" />
+  <!-- Include Tugger definitions -->
+  <xacro:include filename="$(find glr_description)/urdf/glr_tugger.xacro" />
+  <!-- Include Trailer definitions -->
+  <xacro:include filename="$(find glr_description)/urdf/glr_trailer.xacro" />
   <!-- Include Gazebo definitions -->
-  <xacro:include filename="$(find glr_description)/urdf/glr_gazebo.xacro" />
+  <xacro:include filename="$(find glr_description)/urdf/glr_tugger_gazebo.xacro" />
+  <xacro:include filename="$(find glr_description)/urdf/glr_trailer_gazebo.xacro" />
+  <!-- Connection between tugger and trailer -->
+  <joint name="tugger_trailer_joint" type="revolute">
+    <origin xyz="0 0 0" rpy="0 0 0" />
+    <parent link="hitch_link" />
+    <child link="trailer_link" />
+    <axis xyz="0 0 1" />
+    <limit lower="-0.6" upper="0.6" effort="100" velocity="1" />
+    <dynamics damping="0" friction="0" />
+  </joint>
 </robot>

File: urdf/glr_trailer.xacro (robot description, xacro)
@@ -1,8 +1,5 @@
 <?xml version="1.0" encoding="utf-8"?>
-<robot name="glr_description" xmlns:xacro="http://ros.org/wiki/xacro">
-  <!-- Wheel properties -->
-  <xacro:property name="wheel_radius" value="0.1" />
-  <xacro:property name="wheel_width" value="0.08" />
-  <xacro:property name="caster_radius" value="0.08" />
+<robot name="glr_trailer" xmlns:xacro="http://ros.org/wiki/xacro">
+  <!-- Trailer wheel properties -->
   <xacro:property name="trailer_wheel_radius" value="0.1" />
   <xacro:property name="trailer_wheel_width" value="0.08" />
@@ -14,31 +11,23 @@
     <inertia ixx="${1*(2/5) * m * (r*r)}" ixy="0.0" ixz="0.0" iyy="${1*(2/5) * m * (r*r)}" iyz="0.0" izz="${1*(2/5) * m * (r*r)}"/>
   </xacro:macro>
-  <xacro:macro name="cylinder_inertia" params="m r h">
-    <inertial>
-      <mass value="${m}"/>
-      <inertia  ixx="${m*(3*r*r+h*h)/12}" ixy = "0" ixz = "0" iyy="${m*(3*r*r+h*h)/12}" iyz = "0" izz="${m*r*r/2}" />
-    </inertial>
-  </xacro:macro>
-  <!--Robot description  -->
-  <link name="base_link"/>
-  <!-- Robot Footprint -->
-  <link name="base_footprint"/>
-  <joint name="base_joint" type="fixed">
-    <parent link="base_link"/>
-    <child link="base_footprint"/>
-    <origin xyz="0 0 0" rpy="0 0 0"/>
-  </joint>
-  <!-- Tugger -->
-  <link name="chassibigga">
-    <origin xyz="0 0 0" rpy="0 0 0" />
-    <inertial>
-      <origin xyz="0 0 0.155" rpy="0 0 0" />
-      <mass value="555.02" />
-      <xacro:box_inertia m="555.02" w="0.5" d="0.7" h="0.31"/>
-    </inertial>
-    <visual>
-      <origin xyz="0 0 0.155" rpy="0 0 0" />
-      <geometry>
-          <box size="0.50 0.70 0.31"/>
+  <!-- Trailer base link -->
+  <link name="trailer_link">
+    <inertial>
+      <origin rpy="0 0 0" xyz="0.003381 1.5929e-07 0.02162" />
+      <mass value="0.5" />
+      <inertia ixx="1.0" ixy="0.0" ixz="0.0" iyy="1.0" iyz="0.0" izz="1.0" />
+    </inertial>
+  </link>
+  <!-- Connector bar (cambao) -->
+  <link name="cambao">
+    <inertial>
+      <origin xyz="-0.0010213 -0.38489 0.0092469" rpy="0 0 0" />
+      <mass value="1." />
+      <inertia ixx="0.12" ixy="0.0" ixz="0.0" iyy="0.12" iyz="0.0" izz="0.12" />
+    </inertial>
+    <visual>
+      <origin xyz="0 -0.7 0" rpy="0 0 0" />
+     <geometry>
+        <box size="0.1 1.2 0.08"/>
       </geometry>
       <material name="">
@@ -46,131 +35,8 @@
       </material>
     </visual>
-    <collision>
-      <origin xyz="0 0 0.155" rpy="0 0 0" />
-      <geometry>
-          <box size="0.50 0.70 0.31"/>
-      </geometry>
-    </collision>
-  </link>
-  <joint name="base_chassi_joint" type="fixed">
-    <parent link="base_link"/>
-    <child link="chassibigga"/>
-    <origin xyz="0 0 ${wheel_radius}" rpy="0 0 0"/>
-  </joint>
-  <!-- Left Traction Wheel -->
-  <link name="left_wheel">
-    <inertial>
-      <origin xyz="0 0 0" rpy="0 0 0"/>
-      <mass value="12"/>
-      <xacro:sphere_inertia m="12" r="${wheel_radius}"/>
-    </inertial>
-    <visual>
-      <origin xyz="0 0 0" rpy="0 1.5708 0"/>
-      <geometry>
-        <cylinder radius="${wheel_radius}" length="${wheel_width}"/>
-      </geometry>
-      <material name="wheel_material">
-        <color rgba="0.29804 0.29804 0.29804 1"/>
-      </material>
-    </visual>
-    <collision>
-      <origin xyz="0 0 0" rpy="0 1.5708 0"/>
-      <geometry>
-        <cylinder radius="${wheel_radius}" length="${wheel_width}"/>
-      </geometry>
-    </collision>
-  </link>
-  <joint name="left_wheel_joint" type="continuous">
-    <origin xyz="0.25 0 0" rpy="0 0 0"/>
-    <parent link="chassibigga"/>
-    <child link="left_wheel"/>
-    <axis xyz="1 0 0"/>
-    <dynamics damping="0.1" friction="0.1"/>
-  </joint>
-  <!-- Right Traction Wheel -->
-  <link name="right_wheel">
-    <inertial>
-      <origin xyz="0 0 0" rpy="0 0 0"/>
-      <mass value="12"/>
-      <xacro:sphere_inertia m="12" r="${wheel_radius}"/>
-    </inertial>
-    <visual>
-      <origin xyz="0 0 0" rpy="0 1.5708 0"/>
-      <geometry>
-        <cylinder radius="${wheel_radius}" length="${wheel_width}"/>
-      </geometry>
-      <material name="wheel_material">
-        <color rgba="0.29804 0.29804 0.29804 1"/>
-      </material>
-    </visual>
-    <collision>
-      <origin xyz="0 0 0" rpy="0 1.5708 0"/>
-      <geometry>
-        <cylinder radius="${wheel_radius}" length="${wheel_width}"/>
-      </geometry>
-    </collision>
-  </link>
-  <joint name="right_wheel_joint" type="continuous">
-    <origin xyz="-0.25 0 0" rpy="0 0 0"/>
-    <parent link="chassibigga"/>
-    <child link="right_wheel"/>
-    <axis xyz="1 0 0"/>
-    <dynamics damping="0.1" friction="0.1"/>
-  </joint>
-  <!-- ============================================ -->
-  <!-- CASTER WHEELS COMMENTED FOR TESTING -->
-  <!-- ============================================ -->
-  <!--
-  Front/Back Left/Right Caster wheels commented out for testing
-  -->
-  <!-- ============================================ -->
-  <!-- TUGGER-TRAILER CONNECTION -->
-  <!-- ============================================ -->
-  <!-- Hitch point at the back of tugger -->
-  <link name="hitch_link">
-    <inertial>
-      <origin xyz="0 0 0" rpy="0 0 0"/>
-      <mass value="1.0"/>
-      <inertia ixx="0.01" ixy="0" ixz="0" iyy="0.01" iyz="0" izz="0.01"/>
-    </inertial>
-    <visual>
-      <origin xyz="0 0 0" rpy="0 0 0"/>
-      <geometry>
-        <cylinder radius="0.05" length="0.1"/>
-      </geometry>
-      <material name="hitch_material">
-        <color rgba="0.3 0.3 0.3 1"/>
-      </material>
-    </visual>
-    <collision>
-      <origin xyz="0 0 0" rpy="0 0 0"/>
-      <geometry>
-        <cylinder radius="0.05" length="0.1"/>
-      </geometry>
-    </collision>
-  </link>
-  <joint name="hitch_joint" type="fixed">
-    <origin xyz="0 0.35 0.14260" rpy="0 0 0"/>
-    <parent link="chassibigga"/>
-    <child link="hitch_link"/>
-  </joint>
-  <joint name="eixochassibigga" type="revolute">
-    <origin xyz="0 0 0" rpy="0 0 0" />
-    <parent link="hitch_link" />
-    <child link="chassibigga_uni" />
-    <axis xyz="0 0 1" />
-    <limit lower="-0.6" upper="0.6" effort="100" velocity="1" />
-    <dynamics damping="0" friction="0" />
-  </joint>
-  <link name="chassibigga_uni">
-    <inertial>
-      <origin rpy="0 0 0" xyz="0.003381 1.5929e-07 0.02162" />
-      <mass value="0.5" />
-      <inertia ixx="1.0" ixy="0.0" ixz="0.0" iyy="1.0" iyz="0.0" izz="1.0" />
-    </inertial>
-  </link>
-  <joint name="eixochassibigga_cambao" type="revolute">
+  </link>
+  <joint name="trailer_cambao_joint" type="revolute">
     <origin xyz="0 1.1578 0.0112477" rpy="0 0 0" />
-    <parent link="chassibigga_uni" />
+    <parent link="trailer_link" />
     <child link="cambao" />
     <axis xyz="0 1 0" />
@@ -178,22 +44,27 @@
     <dynamics damping="0" friction="0" />
   </joint>
-  <!-- Connector -->
-  <link name="cambao">
-    <inertial>
-      <origin xyz="-0.0010213 -0.38489 0.0092469" rpy="0 0 0" />
-      <mass value="1." />
-      <inertia ixx="0.12" ixy="0.0" ixz="0.0" iyy="0.12" iyz="0.0" izz="0.12" />
-    </inertial>
-    <visual>
-      <origin xyz="0 -0.7 0" rpy="0 0 0" />
+  <!-- Trailer chassis -->
+  <link name="chassi">
+    <inertial>
+      <mass value="80.702" />
+      <xacro:box_inertia m="80.702" w="1" d="1.2" h="0.12"/>
+    </inertial>
+    <visual>
+      <origin xyz="0 0 0.35" rpy="0 0 0" />
      <geometry>
-        <box size="0.1 1.2 0.08"/>
-      </geometry>
-      <material name="">
+        <box size="1 1.2 0.12"/>
+      </geometry>
+      <material name="Cyan">
         <color rgba="0.64706 0.61961 0.58824 1" />
       </material>
     </visual>
-  </link>
-  <joint name="eixocambao_chassi" type="revolute">
+    <collision>
+      <origin xyz="0 0 0.43" rpy="0 0 0" />
+      <geometry>
+        <box size="1 1.2 0.12"/>
+      </geometry>
+    </collision>
+  </link>
+  <joint name="cambao_chassi_joint" type="revolute">
     <origin xyz="0 0.445 -0.31525" rpy="0 0 0" />
     <parent link="cambao" />
@@ -203,27 +74,6 @@
     <dynamics damping="0" friction="0" />
   </joint>
-  <!-- Trailer -->
-  <link name="chassi">
-    <inertial>
-      <mass value="80.702" />
-      <xacro:box_inertia m="80.702" w="1" d="1.2" h="0.12"/>
-    </inertial>
-    <visual>
-      <origin xyz="0 0 0.35" rpy="0 0 0" />
-     <geometry>
-        <box size="1 1.2 0.12"/>
-      </geometry>
-      <material name="Cyan">
-        <color rgba="0.64706 0.61961 0.58824 1" />
-      </material>
-    </visual>
-    <collision>
-      <origin xyz="0 0 0.43" rpy="0 0 0" />
-      <geometry>
-        <box size="1 1.2 0.12"/>
-      </geometry>
-    </collision>
-  </link>
-  <!-- Trailer wheel mounts -->
+  <!-- Trailer wheel mounts and wheels -->
+  <!-- Front Left -->
   <link name="rodeirodiant1">
     <inertial>
@@ -270,4 +120,5 @@
     <dynamics damping="0" friction="10.0" />
   </joint>
+  <!-- Front Right -->
   <link name="rodeirodiant2">
     <inertial>
@@ -314,4 +165,5 @@
     <dynamics damping="0" friction="10.0" />
   </joint>
+  <!-- Rear Left -->
   <link name="rodeirotras1">
     <inertial>
@@ -358,4 +210,5 @@
     <dynamics damping="0" friction="10.0" />
   </joint>
+  <!-- Rear Right -->
   <link name="rodeirotras2">
     <inertial>
@@ -402,31 +255,3 @@
     <dynamics damping="0" friction="10.0" />
   </joint>
-  <!-- Generic LiDAR -->
-  <link name="lidar_link">
-    <inertial>
-      <origin xyz="0 0 0" rpy="0 0 0"/>
-      <mass value="0.5"/>
-      <inertia ixx="0.001" ixy="0" ixz="0" iyy="0.001" iyz="0" izz="0.001"/>
-    </inertial>
-    <visual>
-      <origin xyz="0 0 0" rpy="0 0 0"/>
-      <geometry>
-        <cylinder radius="0.05" length="0.07"/>
-      </geometry>
-      <material name="lidar_material">
-        <color rgba="0.2 0.2 0.2 1"/>
-      </material>
-    </visual>
-    <collision>
-      <origin xyz="0 0 0" rpy="0 0 0"/>
-      <geometry>
-        <cylinder radius="0.05" length="0.07"/>
-      </geometry>
-    </collision>
-  </link>
-  <joint name="lidar_joint" type="fixed">
-    <parent link="chassibigga"/>
-    <child link="lidar_link"/>
-    <origin xyz="0 -0.25 0.34" rpy="0 0 0"/>
-  </joint>
 </robot>

File: urdf/glr_trailer_gazebo.xacro (robot description, xacro)
@@ -1,23 +1,7 @@
 <?xml version="1.0" encoding="utf-8"?>
-<robot name="glr_gazebo" xmlns:xacro="http://ros.org/wiki/xacro">
+<robot name="glr_trailer_gazebo" xmlns:xacro="http://ros.org/wiki/xacro">
   <!-- ============================================ -->
-  <!-- GAZEBO MATERIAL DEFINITIONS -->
+  <!-- TRAILER GAZEBO MATERIAL DEFINITIONS -->
   <!-- ============================================ -->
-  <gazebo reference="chassibigga">
-    <material>Gazebo/Orange</material>
-  </gazebo>
-  <gazebo reference="left_wheel">
-    <material>Gazebo/Black</material>
-    <mu1>1.0</mu1>
-    <mu2>1.0</mu2>
-  </gazebo>
-  <gazebo reference="right_wheel">
-    <material>Gazebo/Black</material>
-    <mu1>1.0</mu1>
-    <mu2>1.0</mu2>
-  </gazebo>
-  <gazebo reference="hitch_link">
-    <material>Gazebo/DarkGrey</material>
-  </gazebo>
   <gazebo reference="cambao">
     <material>Gazebo/Grey</material>
@@ -49,66 +33,4 @@
   <gazebo reference="rodatras2">
     <material>Gazebo/Black</material>
-  </gazebo>
-  <!-- ============================================ -->
-  <!-- DIFFERENTIAL DRIVE PLUGIN -->
-  <!-- ============================================ -->
-  <gazebo>
-    <plugin name="differential_drive_controller" filename="libgazebo_ros_diff_drive.so">
-      <ros>
-        <remapping>cmd_vel:=cmd_vel</remapping>
-        <remapping>odom:=odom</remapping>
-      </ros>
-      <update_rate>100.0</update_rate>
-      <left_joint>left_wheel_joint</left_joint>
-      <right_joint>right_wheel_joint</right_joint>
-      <wheel_separation>0.5</wheel_separation>
-      <wheel_diameter>0.2</wheel_diameter>
-      <max_wheel_torque>200</max_wheel_torque>
-      <max_wheel_acceleration>10.0</max_wheel_acceleration>
-      <publish_odom>true</publish_odom>
-      <publish_odom_tf>true</publish_odom_tf>
-      <publish_wheel_tf>true</publish_wheel_tf>
-      <odometry_frame>odom</odometry_frame>
-      <robot_base_frame>base_link</robot_base_frame>
-    </plugin>
-  </gazebo>
-  <!-- ============================================ -->
-  <!-- LIDAR SENSOR PLUGIN -->
-  <!-- ============================================ -->
-  <gazebo reference="lidar_link">
-    <material>Gazebo/DarkGrey</material>
-    <sensor type="ray" name="lidar_sensor">
-      <pose>0 0 0 0 0 0</pose>
-      <visualize>false</visualize>
-      <update_rate>10</update_rate>
-      <ray>
-        <scan>
-          <horizontal>
-            <samples>360</samples>
-            <resolution>1</resolution>
-            <min_angle>-3.14159</min_angle>
-            <max_angle>3.14159</max_angle>
-          </horizontal>
-        </scan>
-        <range>
-          <min>0.1</min>
-          <max>30.0</max>
-          <resolution>0.01</resolution>
-        </range>
-        <noise>
-          <type>gaussian</type>
-          <mean>0.0</mean>
-          <stddev>0.01</stddev>
-        </noise>
-      </ray>
-      <plugin name="gazebo_ros_lidar" filename="libgazebo_ros_ray_sensor.so">
-        <ros>
-          <namespace>/glr_description</namespace>
-          <remapping>~/out:=scan</remapping>
-        </ros>
-        <output_type>sensor_msgs/LaserScan</output_type>
-        <frame_name>lidar_link</frame_name>
-      </plugin>
-    </sensor>
   </gazebo>
   <!-- ============================================ -->

Commit message: :construction: trying to create the first map

File: urdf/glr.xacro (robot description, xacro)
@@ -1,10 +1,8 @@
 <?xml version="1.0" encoding="utf-8"?>
 <robot name="glr_description" xmlns:xacro="http://ros.org/wiki/xacro">
-  <!-- Include Tugger definitions -->
   <xacro:include filename="$(find glr_description)/urdf/glr_tugger.xacro" />
-  <!-- Include Trailer definitions -->
+  <xacro:include filename="$(find glr_description)/urdf/glr_tugger_gazebo.xacro" />
+  <xacro:include filename="$(find glr_description)/ros2_control/glr_ros2_control.xacro" />
   <xacro:include filename="$(find glr_description)/urdf/glr_trailer.xacro" />
-  <!-- Include Gazebo definitions -->
-  <xacro:include filename="$(find glr_description)/urdf/glr_tugger_gazebo.xacro" />
   <xacro:include filename="$(find glr_description)/urdf/glr_trailer_gazebo.xacro" />
   <!-- Connection between tugger and trailer -->

File: urdf/glr_trailer.xacro (robot description, xacro)
@@ -45,5 +45,5 @@
   </joint>
   <!-- Trailer chassis -->
-  <link name="chassi">
+  <link name="trailer_footprint">
     <inertial>
       <mass value="80.702" />
@@ -69,5 +69,5 @@
     <origin xyz="0 0.445 -0.31525" rpy="0 0 0" />
     <parent link="cambao" />
-    <child link="chassi" />
+    <child link="trailer_footprint" />
     <axis xyz="0 0 1" />
     <limit lower="-0.4" upper="0.4" effort="100" velocity="1" />
@@ -85,5 +85,5 @@
   <joint name="eixorodeirodiant1" type="revolute">
     <origin xyz="0.39 -0.445 0.36525" rpy="0 0 0" />
-    <parent link="chassi" />
+    <parent link="trailer_footprint" />
     <child link="rodeirodiant1" />
     <axis xyz="0 0 1" />
@@ -130,5 +130,5 @@
   <joint name="eixorodeirodiant2" type="revolute">
     <origin xyz="-0.39 -0.445 0.36525" rpy="0 0 0" />
-    <parent link="chassi" />
+    <parent link="trailer_footprint" />
     <child link="rodeirodiant2" />
     <axis xyz="0 0 1" />
@@ -175,5 +175,5 @@
   <joint name="eixorodeirotras1" type="revolute">
     <origin xyz="0.39 0.445 0.36525" rpy="0 0 0" />
-    <parent link="chassi" />
+    <parent link="trailer_footprint" />
     <child link="rodeirotras1" />
     <axis xyz="0 0 1" />
@@ -220,5 +220,5 @@
   <joint name="eixorodeirotras2" type="revolute">
     <origin xyz="-0.39 0.445 0.36525" rpy="0 0 0" />
-    <parent link="chassi" />
+    <parent link="trailer_footprint" />
     <child link="rodeirotras2" />
     <axis xyz="0 0 1" />

File: urdf/glr_trailer_gazebo.xacro (robot description, xacro)
@@ -7,5 +7,5 @@
     <material>Gazebo/Grey</material>
   </gazebo>
-  <gazebo reference="chassi">
+  <gazebo reference="trailer_footprint">
     <material>Gazebo/Orange</material>
   </gazebo>

Commit message: :construction: with base_footprint error

File: urdf/glr.xacro (robot description, xacro)
@@ -4,8 +4,8 @@
   <xacro:include filename="$(find glr_description)/urdf/glr_tugger_gazebo.xacro" />
   <xacro:include filename="$(find glr_description)/ros2_control/glr_ros2_control.xacro" />
-  <xacro:include filename="$(find glr_description)/urdf/glr_trailer.xacro" />
-  <xacro:include filename="$(find glr_description)/urdf/glr_trailer_gazebo.xacro" />
+  <!-- <xacro:include filename="$(find glr_description)/urdf/glr_trailer.xacro" /> -->
+  <!-- <xacro:include filename="$(find glr_description)/urdf/glr_trailer_gazebo.xacro" />   -->
   <!-- Connection between tugger and trailer -->
-  <joint name="tugger_trailer_joint" type="revolute">
+  <!-- <joint name="tugger_trailer_joint" type="revolute">
     <origin xyz="0 0 0" rpy="0 0 0" />
     <parent link="hitch_link" />
@@ -14,4 +14,4 @@
     <limit lower="-0.6" upper="0.6" effort="100" velocity="1" />
     <dynamics damping="0" friction="0" />
-  </joint>
+  </joint> -->
 </robot>

File: urdf/glr_tugger_gazebo.xacro (robot description, xacro)
@@ -1,7 +1,5 @@
-<?xml version="1.0" encoding="utf-8"?>
-<robot name="glr_tugger_gazebo" xmlns:xacro="http://ros.org/wiki/xacro">
-  <!-- ============================================ -->
-  <!-- TUGGER GAZEBO MATERIAL DEFINITIONS -->
-  <!-- ============================================ -->
+<?xml version="1.0"?>
+<robot xmlns:xacro="http://ros.org/wiki/xacro">
+  <!-- Materiais e parâmetros do Gazebo -->
   <gazebo reference="base_link">
     <material>Gazebo/Orange</material>
@@ -17,70 +15,28 @@
     <mu2>1.0</mu2>
   </gazebo>
-  <gazebo reference="hitch_link">
-    <material>Gazebo/DarkGrey</material>
-  </gazebo>
-  <gazebo reference="lidar_link">
-    <material>Gazebo/DarkGrey</material>
-  </gazebo>
-  <!-- ============================================ -->
-  <!-- DIFFERENTIAL DRIVE PLUGIN -->
-  <!-- ============================================ -->
+  <!-- =========================== -->
+  <!-- ROS 2 CONTROL - GazeboSystem -->
+  <!-- =========================== -->
   <gazebo>
-    <plugin name="differential_drive_controller" filename="libgazebo_ros_diff_drive.so">
-      <ros>
-        <remapping>cmd_vel:=cmd_vel</remapping>
-        <remapping>odom:=odom</remapping>
-      </ros>
-      <update_rate>100.0</update_rate>
-      <left_joint>left_wheel_joint</left_joint>
-      <right_joint>right_wheel_joint</right_joint>
-      <wheel_separation>0.5</wheel_separation>
-      <wheel_diameter>0.2</wheel_diameter>
-      <max_wheel_torque>200</max_wheel_torque>
-      <max_wheel_acceleration>10.0</max_wheel_acceleration>
-      <publish_odom>true</publish_odom>
-      <publish_odom_tf>true</publish_odom_tf>
-      <publish_wheel_tf>true</publish_wheel_tf>
-      <odometry_frame>odom</odometry_frame>
-      <robot_base_frame>base_link</robot_base_frame>
+    <plugin filename="libgazebo_ros2_control.so" name="gazebo_ros2_control">
+      <ros2_control name="glr_system" type="system">
+        <hardware>
+          <plugin>gazebo_ros2_control/GazeboSystem</plugin>
+          <param name="command_interfaces">["velocity"]</param>
+          <param name="state_interfaces">["position","velocity"]</param>
+        </hardware>
+        <!-- Repete os joints aqui dentro -->
+        <joint name="left_wheel_joint">
+          <command_interface name="velocity"/>
+          <state_interface name="position"/>
+          <state_interface name="velocity"/>
+        </joint>
+        <joint name="right_wheel_joint">
+          <command_interface name="velocity"/>
+          <state_interface name="position"/>
+          <state_interface name="velocity"/>
+        </joint>
+      </ros2_control>
     </plugin>
   </gazebo>
-  <!-- ============================================ -->
-  <!-- LIDAR SENSOR PLUGIN -->
-  <!-- ============================================ -->
-  <gazebo reference="lidar_link">
-    <sensor type="ray" name="lidar_sensor">
-      <pose>0 0 0 0 0 0</pose>
-      <visualize>false</visualize>
-      <update_rate>10</update_rate>
-      <ray>
-        <scan>
-          <horizontal>
-            <samples>360</samples>
-            <resolution>1</resolution>
-            <min_angle>-3.14159</min_angle>
-            <max_angle>3.14159</max_angle>
-          </horizontal>
-        </scan>
-        <range>
-          <min>0.1</min>
-          <max>30.0</max>
-          <resolution>0.01</resolution>
-        </range>
-        <noise>
-          <type>gaussian</type>
-          <mean>0.0</mean>
-          <stddev>0.01</stddev>
-        </noise>
-      </ray>
-      <plugin name="gazebo_ros_lidar" filename="libgazebo_ros_ray_sensor.so">
-        <ros>
-          <namespace>/glr_description</namespace>
-          <remapping>~/out:=scan</remapping>
-        </ros>
-        <output_type>sensor_msgs/LaserScan</output_type>
-        <frame_name>lidar_link</frame_name>
-      </plugin>
-    </sensor>
-  </gazebo>
 </robot>
