Commit message: :construction: fixing trailer moviment

File: urdf/glr.urdf (robot description, URDF)
Before this commit: robot glr_tugger, 11 links, 10 joints
Links:
- added link cambao, mass 1.0; collision box size=0.05 0.6 0.08; visual box size=0.05 0.6 0.08
- added link chassi, mass 80.702; collision box size=1 1.2 0.12; visual box size=1 1.2 0.12
- added link rodadiant1, mass 2; collision cylinder length=0.08 radius=0.1; visual cylinder length=0.08 radius=0.1
- added link rodadiant2, mass 2; collision cylinder length=0.08 radius=0.1; visual cylinder length=0.08 radius=0.1
- added link rodatras1, mass 2; collision cylinder length=0.08 radius=0.1; visual cylinder length=0.08 radius=0.1
- added link rodatras2, mass 2; collision cylinder length=0.08 radius=0.1; visual cylinder length=0.08 radius=0.1
- added link rodeirodiant1, mass 0.5
- added link rodeirodiant2, mass 0.5
- added link rodeirotras1, mass 0.5
- added link rodeirotras2, mass 0.5
- added link trailer_link, mass 0.5
Joints:
- added joint cambao_chassi_joint: type revolute, parent cambao, child chassi, origin xyz=0 0.6 -0.284 rpy=0 0 0, axis 0 0 1, limit lower=-0.8 upper=0.8 effort=100 velocity=1
- added joint eixorodadiant1: type continuous, parent rodeirodiant1, child rodadiant1, origin xyz=0.08 0 -0.22125 rpy=0 0 0, axis 1 0 0
- added joint eixorodadiant2: type continuous, parent rodeirodiant2, child rodadiant2, origin xyz=-0.08 0 -0.22125 rpy=0 0 0, axis 1 0 0
- added joint eixorodatras1: type continuous, parent rodeirotras1, child rodatras1, origin xyz=0.08 0 -0.22125 rpy=0 0 0, axis 1 0 0
- added joint eixorodatras2: type continuous, parent rodeirotras2, child rodatras2, origin xyz=-0.08 0 -0.22125 rpy=0 0 0, axis 1 0 0
- added joint eixorodeirodiant1: type continuous, parent chassi, child rodeirodiant1, origin xyz=0.39 0.155 0.36525 rpy=0 0 0, axis 0 0 1
- added joint eixorodeirodiant2: type continuous, parent chassi, child rodeirodiant2, origin xyz=-0.39 0.155 0.36525 rpy=0 0 0, axis 0 0 1
- added joint eixorodeirotras1: type continuous, parent chassi, child rodeirotras1, origin xyz=0.39 1.045 0.36525 rpy=0 0 0, axis 0 0 1
- added joint eixorodeirotras2: type continuous, parent chassi, child rodeirotras2, origin xyz=-0.39 1.045 0.36525 rpy=0 0 0, axis 0 0 1
- added joint trailer_cambao_joint: type revolute, parent trailer_link, child cambao, origin xyz=0 0 0 rpy=0 0 0, axis 0 0 1, limit lower=-1.57 upper=1.57 effort=100 velocity=1
- added joint tugger_trailer_joint: type revolute, parent hitch_link, child trailer_link, origin xyz=0 0 0 rpy=0 0 0, axis 0 0 1, limit lower=-0.6 upper=0.6 effort=100 velocity=1

File: urdf/glr.xacro (robot description, xacro)
@@ -5,7 +5,4 @@
   <!-- Include Trailer definitions -->
   <xacro:include filename="$(find glr_description)/urdf/glr_trailer.xacro" />
-  <!-- Include Gazebo definitions -->
-  <xacro:include filename="$(find glr_description)/urdf/glr_tugger_gazebo.xacro" />
-  <xacro:include filename="$(find glr_description)/urdf/glr_trailer_gazebo.xacro" />
   <!-- Connection between tugger and trailer -->
   <joint name="tugger_trailer_joint" type="revolute">

File: urdf/glr_trailer.xacro (robot description, xacro)
@@ -1,64 +1,66 @@
 <?xml version="1.0" encoding="utf-8"?>
 <robot name="glr_trailer" xmlns:xacro="http://ros.org/wiki/xacro">
-  <!-- Trailer wheel properties -->
   <xacro:property name="trailer_wheel_radius" value="0.1" />
   <xacro:property name="trailer_wheel_width" value="0.08" />
-  <!-- Define intertial property macros  -->
   <xacro:macro name="box_inertia" params="m w d h">
-    <inertia ixx="${1*(m/12) * (h*h + d*d)}" ixy="0.0" ixz="0.0" iyy="${1*(m/12) * (w*w + d*d)}" iyz="0.0" izz="${1*(m/12) * (w*w + h*h)}"/>
+    <inertia ixx="${(m/12) * (h*h + d*d)}" ixy="0.0" ixz="0.0" iyy="${(m/12) * (w*w + d*d)}" iyz="0.0" izz="${(m/12) * (w*w + h*h)}"/>
   </xacro:macro>
   <xacro:macro name="sphere_inertia" params="m r">
-    <inertia ixx="${1*(2/5) * m * (r*r)}" ixy="0.0" ixz="0.0" iyy="${1*(2/5) * m * (r*r)}" iyz="0.0" izz="${1*(2/5) * m * (r*r)}"/>
+    <inertia ixx="${(2/5) * m * (r*r)}" ixy="0.0" ixz="0.0" iyy="${(2/5) * m * (r*r)}" iyz="0.0" izz="${(2/5) * m * (r*r)}"/>
   </xacro:macro>
-  <!-- Trailer base link -->
   <link name="trailer_link">
     <inertial>
-      <origin rpy="0 0 0" xyz="0.003381 1.5929e-07 0.02162" />
-      <mass value="0.5" />
-      <inertia ixx="1.0" ixy="0.0" ixz="0.0" iyy="1.0" iyz="0.0" izz="1.0" />
-    </inertial>
-  </link>
-  <!-- Connector bar (cambao) -->
+      <origin rpy="0 0 0" xyz="0 0 0" />
+      <mass value="0.5" />
+      <inertia ixx="0.01" ixy="0.0" ixz="0.0" iyy="0.01" iyz="0.0" izz="0.01" />
+    </inertial>
+  </link>
   <link name="cambao">
     <inertial>
-      <origin xyz="-0.0010213 -0.38489 0.0092469" rpy="0 0 0" />
-      <mass value="1." />
-      <inertia ixx="0.12" ixy="0.0" ixz="0.0" iyy="0.12" iyz="0.0" izz="0.12" />
-    </inertial>
-    <visual>
-      <origin xyz="0 -0.7 0" rpy="0 0 0" />
-     <geometry>
-        <box size="0.1 1.2 0.08"/>
-      </geometry>
-      <material name="">
-        <color rgba="0.64706 0.61961 0.58824 1" />
+      <origin xyz="0 0.3 0" rpy="0 0 0" />
+      <mass value="1.0" />
+      <inertia ixx="0.03" ixy="0.0" ixz="0.0" iyy="0.001" iyz="0.0" izz="0.03" />
+    </inertial>
+    <visual>
+      <origin xyz="0 0.3 0" rpy="0 0 0" />
+      <geometry>
+        <box size="0.05 0.6 0.08"/>
+      </geometry>
+      <material name="Grey">
+        <color rgba="0.6 0.6 0.6 1" />
       </material>
     </visual>
+    <collision>
+      <origin xyz="0 0.3 0" rpy="0 0 0" />
+      <geometry>
+        <box size="0.05 0.6 0.08"/>
+      </geometry>
+    </collision>
   </link>
   <joint name="trailer_cambao_joint" type="revolute">
-    <origin xyz="0 1.1578 0.0112477" rpy="0 0 0" />
+    <origin xyz="0 0 0" rpy="0 0 0" />
     <parent link="trailer_link" />
     <child link="cambao" />
-    <axis xyz="0 1 0" />
-    <limit lower="-0.6" upper="0.6" effort="100" velocity="1" />
-    <dynamics damping="0" friction="0" />
-  </joint>
-  <!-- Trailer chassis -->
+    <axis xyz="0 0 1" />
+    <limit lower="-1.57" upper="1.57" effort="100" velocity="1" />
+    <dynamics damping="10000.0" friction="0.0" />
+  </joint>
   <link name="chassi">
     <inertial>
+      <origin xyz="0 0.6 0.35" rpy="0 0 0" />
       <mass value="80.702" />
       <xacro:box_inertia m="80.702" w="1" d="1.2" h="0.12"/>
     </inertial>
     <visual>
-      <origin xyz="0 0 0.35" rpy="0 0 0" />
-     <geometry>
+      <origin xyz="0 0.6 0.35" rpy="0 0 0" />
+      <geometry>
         <box size="1 1.2 0.12"/>
       </geometry>
       <material name="Cyan">
-        <color rgba="0.64706 0.61961 0.58824 1" />
+        <color rgba="0 1 1 1" />
       </material>
     </visual>
     <collision>
-      <origin xyz="0 0 0.43" rpy="0 0 0" />
+      <origin xyz="0 0.6 0.35" rpy="0 0 0" />
       <geometry>
         <box size="1 1.2 0.12"/>
@@ -67,27 +69,24 @@
   </link>
   <joint name="cambao_chassi_joint" type="revolute">
-    <origin xyz="0 0.445 -0.31525" rpy="0 0 0" />
+    <origin xyz="0 0.6 -0.284" rpy="0 0 0" />
     <parent link="cambao" />
     <child link="chassi" />
     <axis xyz="0 0 1" />
-    <limit lower="-0.4" upper="0.4" effort="100" velocity="1" />
-    <dynamics damping="0" friction="0" />
-  </joint>
-  <!-- Trailer wheel mounts and wheels -->
-  <!-- Front Left -->
+    <limit lower="-0.8" upper="0.8" effort="100" velocity="1" />
+    <dynamics damping="10000.0" friction="0.0" />
+  </joint>
   <link name="rodeirodiant1">
     <inertial>
-      <origin xyz="-0.010304 0.018687 -0.067271" rpy="0 0 0" />
-      <mass value="0.5" />
-      <inertia ixx="0.11" ixy="0.0" ixz="0.0" iyy="0.11" iyz="0.0" izz="0.11" />
-    </inertial>
-  </link>
-  <joint name="eixorodeirodiant1" type="revolute">
-    <origin xyz="0.39 -0.445 0.36525" rpy="0 0 0" />
+      <origin xyz="0 0 0" rpy="0 0 0" />
+      <mass value="0.5" />
+      <inertia ixx="0.01" ixy="0.0" ixz="0.0" iyy="0.01" iyz="0.0" izz="0.01" />
+    </inertial>
+  </link>
+  <joint name="eixorodeirodiant1" type="continuous">
+    <origin xyz="0.39 0.155 0.36525" rpy="0 0 0" />
     <parent link="chassi" />
     <child link="rodeirodiant1" />
     <axis xyz="0 0 1" />
-    <limit lower="-1" upper="1" effort="100" velocity="1" />
-    <dynamics damping="0" friction="10.0" />
+    <dynamics damping="0.0" friction="0.0" />
   </joint>
   <link name="rodadiant1">
@@ -102,7 +101,4 @@
         <cylinder radius="${trailer_wheel_radius}" length="${trailer_wheel_width}"/>
       </geometry>
-      <material name="">
-        <color rgba="0.29804 0.29804 0.29804 1" />
-      </material>
     </visual>
     <collision>
@@ -118,21 +114,19 @@
     <child link="rodadiant1" />
     <axis xyz="1 0 0" />
-    <dynamics damping="0" friction="10.0" />
-  </joint>
-  <!-- Front Right -->
+    <dynamics damping="0.0" friction="0.0" />
+  </joint>
   <link name="rodeirodiant2">
     <inertial>
-      <origin xyz="0.010304 0.018687 -0.067271" rpy="0 0 0" />
-      <mass value="0.5" />
-      <inertia ixx="0.011" ixy="0.0" ixz="0.0" iyy="0.011" iyz="0.0" izz="0.11" />
-    </inertial>
-  </link>
-  <joint name="eixorodeirodiant2" type="revolute">
-    <origin xyz="-0.39 -0.445 0.36525" rpy="0 0 0" />
+      <origin xyz="0 0 0" rpy="0 0 0" />
+      <mass value="0.5" />
+      <inertia ixx="0.01" ixy="0.0" ixz="0.0" iyy="0.01" iyz="0.0" izz="0.01" />
+    </inertial>
+  </link>
+  <joint name="eixorodeirodiant2" type="continuous">
+    <origin xyz="-0.39 0.155 0.36525" rpy="0 0 0" />
     <parent link="chassi" />
     <child link="rodeirodiant2" />
     <axis xyz="0 0 1" />
-    <limit lower="-0.7" upper="0.7" effort="100" velocity="1" />
-    <dynamics damping="0" friction="1.0" />
+    <dynamics damping="0.0" friction="0.0" />
   </joint>
   <link name="rodadiant2">
@@ -147,7 +141,4 @@
         <cylinder radius="${trailer_wheel_radius}" length="${trailer_wheel_width}"/>
       </geometry>
-      <material name="">
-        <color rgba="0.29804 0.29804 0.29804 1" />
-      </material>
     </visual>
     <collision>
@@ -163,21 +154,19 @@
     <child link="rodadiant2" />
     <axis xyz="1 0 0" />
-    <dynamics damping="0" friction="10.0" />
-  </joint>
-  <!-- Rear Left -->
+    <dynamics damping="0.0" friction="0.0" />
+  </joint>
   <link name="rodeirotras1">
     <inertial>
-      <origin xyz="-0.014075 -2.2041E-06 -0.076225" rpy="0 0 0" />
-      <mass value="0.5" />
-      <inertia ixx="0.11" ixy="0.0" ixz="0.0" iyy="0.11" iyz="0.0" izz="0.11" />
-    </inertial>
-  </link>
-  <joint name="eixorodeirotras1" type="revolute">
-    <origin xyz="0.39 0.445 0.36525" rpy="0 0 0" />
+      <origin xyz="0 0 0" rpy="0 0 0" />
+      <mass value="0.5" />
+      <inertia ixx="0.01" ixy="0.0" ixz="0.0" iyy="0.01" iyz="0.0" izz="0.01" />
+    </inertial>
+  </link>
+  <joint name="eixorodeirotras1" type="continuous">
+    <origin xyz="0.39 1.045 0.36525" rpy="0 0 0" />
     <parent link="chassi" />
     <child link="rodeirotras1" />
     <axis xyz="0 0 1" />
-    <limit lower="-1" upper="1" effort="100" velocity="1" />
-    <dynamics damping="0" friction="10.0" />
+    <dynamics damping="0.0" friction="0.0" />
   </joint>
   <link name="rodatras1">
@@ -192,7 +181,4 @@
         <cylinder radius="${trailer_wheel_radius}" length="${trailer_wheel_width}"/>
       </geometry>
-      <material name="">
-        <color rgba="0.29804 0.29804 0.29804 1" />
-      </material>
     </visual>
     <collision>
@@ -204,25 +190,23 @@
   </link>
   <joint name="eixorodatras1" type="continuous">
-    <origin xyz="0.080 0 -0.22125" rpy="0 0 0" />
+    <origin xyz="0.08 0 -0.22125" rpy="0 0 0" />
     <parent link="rodeirotras1" />
     <child link="rodatras1" />
     <axis xyz="1 0 0" />
-    <dynamics damping="0" friction="10.0" />
-  </joint>
-  <!-- Rear Right -->
+    <dynamics damping="0.0" friction="0.0" />
+  </joint>
   <link name="rodeirotras2">
     <inertial>
-      <origin xyz="0.014075 -2.2041E-06 -0.076225" rpy="0 0 0" />
-      <mass value="0.5" />
-      <inertia ixx="0.11" ixy="0.0" ixz="0.0" iyy="0.11" iyz="0.0" izz="0.11" />
-    </inertial>
-  </link>
-  <joint name="eixorodeirotras2" type="revolute">
-    <origin xyz="-0.39 0.445 0.36525" rpy="0 0 0" />
+      <origin xyz="0 0 0" rpy="0 0 0" />
+      <mass value="0.5" />
+      <inertia ixx="0.01" ixy="0.0" ixz="0.0" iyy="0.01" iyz="0.0" izz="0.01" />
+    </inertial>
+  </link>
+  <joint name="eixorodeirotras2" type="continuous">
+    <origin xyz="-0.39 1.045 0.36525" rpy="0 0 0" />
     <parent link="chassi" />
     <child link="rodeirotras2" />
     <axis xyz="0 0 1" />
-    <limit lower="-1" upper="1" effort="100" velocity="1" />
-    <dynamics damping="0" friction="10.0" />
+    <dynamics damping="0.0" friction="0.0" />
   </joint>
   <link name="rodatras2">
@@ -237,7 +221,4 @@
         <cylinder radius="${trailer_wheel_radius}" length="${trailer_wheel_width}"/>
       </geometry>
-      <material name="">
-        <color rgba="0.29804 0.29804 0.29804 1" />
-      </material>
     </visual>
     <collision>
@@ -249,9 +230,9 @@
   </link>
   <joint name="eixorodatras2" type="continuous">
-    <origin xyz="-0.080 0 -0.22125" rpy="0 0 0" />
+    <origin xyz="-0.08 0 -0.22125" rpy="0 0 0" />
     <parent link="rodeirotras2" />
     <child link="rodatras2" />
     <axis xyz="1 0 0" />
-    <dynamics damping="0" friction="10.0" />
+    <dynamics damping="0.0" friction="0.0" />
   </joint>
 </robot>

File: urdf/glr_tugger.xacro (robot description, xacro)
@@ -4,5 +4,13 @@
   <xacro:property name="wheel_radius" value="0.1" />
   <xacro:property name="wheel_width" value="0.08" />
-  <xacro:property name="caster_radius" value="0.08" />
+  <xacro:property name="wheel_mass" value="12" />
+  <!-- Caster properties -->
+  <xacro:property name="caster_radius" value="0.05" />
+  <xacro:property name="caster_x" value="0.20" />
+  <xacro:property name="caster_y" value="0.28" />
+  <xacro:property name="caster_z" value="-0.05" />
+  <xacro:property name="chassi_z" value="0.1" />
+  <xacro:property name="lidar_offset_z" value="0.185" />
+  <xacro:property name="hitch_offset_z" value="0.04" />
   <!-- Define intertial property macros  -->
   <xacro:macro name="box_inertia" params="m w d h">
@@ -19,5 +27,11 @@
   </xacro:macro>
   <!--Robot description  -->
-  <link name="base_link"/>
+  <link name="base_link">
+    <inertial>
+      <origin xyz="0 0 0" rpy="0 0 0"/>
+      <mass value="0.1"/>
+      <inertia ixx="0.0001" ixy="0" ixz="0" iyy="0.0001" iyz="0" izz="0.0001"/>
+    </inertial>
+  </link>
   <!-- Robot Footprint -->
   <link name="base_footprint"/>
@@ -31,10 +45,10 @@
     <origin xyz="0 0 0" rpy="0 0 0" />
     <inertial>
-      <origin xyz="0 0 0.155" rpy="0 0 0" />
-      <mass value="555.02" />
-      <xacro:box_inertia m="555.02" w="0.5" d="0.7" h="0.31"/>
-    </inertial>
-    <visual>
-      <origin xyz="0 0 0.155" rpy="0 0 0" />
+      <origin xyz="0 0 ${chassi_z}" rpy="0 0 0" />
+      <mass value="40" />
+      <xacro:box_inertia m="40" w="0.5" d="0.7" h="0.31"/>
+    </inertial>
+    <visual>
+      <origin xyz="0 0 ${chassi_z}" rpy="0 0 0" />
       <geometry>
           <box size="0.50 0.70 0.31"/>
@@ -45,5 +59,5 @@
     </visual>
     <collision>
-      <origin xyz="0 0 0.155" rpy="0 0 0" />
+      <origin xyz="0 0 ${chassi_z}" rpy="0 0 0" />
       <geometry>
           <box size="0.50 0.70 0.31"/>
@@ -60,6 +74,10 @@
     <inertial>
       <origin xyz="0 0 0" rpy="0 0 0"/>
-      <mass value="12"/>
-      <xacro:sphere_inertia m="12" r="${wheel_radius}"/>
+      <mass value="${wheel_mass}"/>
+      <inertia ixx="${0.5 * wheel_mass * wheel_radius * wheel_radius}"
+               ixy="0" ixz="0"
+               iyy="${(1.0/12.0) * wheel_mass * (3 * wheel_radius * wheel_radius + wheel_width * wheel_width)}"
+               iyz="0"
+               izz="${(1.0/12.0) * wheel_mass * (3 * wheel_radius * wheel_radius + wheel_width * wheel_width)}"/>
     </inertial>
     <visual>
@@ -84,5 +102,5 @@
     <child link="left_wheel"/>
     <axis xyz="1 0 0"/>
-    <dynamics damping="0.1" friction="0.1"/>
+    <dynamics damping="0.5" friction="1.0"/>
   </joint>
   <!-- Right Traction Wheel -->
@@ -90,6 +108,10 @@
     <inertial>
       <origin xyz="0 0 0" rpy="0 0 0"/>
-      <mass value="12"/>
-      <xacro:sphere_inertia m="12" r="${wheel_radius}"/>
+      <mass value="${wheel_mass}"/>
+      <inertia ixx="${0.5 * wheel_mass * wheel_radius * wheel_radius}"
+               ixy="0" ixz="0"
+               iyy="${(1.0/12.0) * wheel_mass * (3 * wheel_radius * wheel_radius + wheel_width * wheel_width)}"
+               iyz="0"
+               izz="${(1.0/12.0) * wheel_mass * (3 * wheel_radius * wheel_radius + wheel_width * wheel_width)}"/>
     </inertial>
     <visual>
@@ -114,9 +136,44 @@
     <child link="right_wheel"/>
     <axis xyz="1 0 0"/>
-    <dynamics damping="0.1" friction="0.1"/>
+    <dynamics damping="0.5" friction="1.0"/>
   </joint>
   <!-- ============================================ -->
-  <!-- CASTER WHEELS COMMENTED FOR TESTING -->
+  <!-- CASTER WHEELS -->
   <!-- ============================================ -->
+  <xacro:macro name="caster_wheel" params="prefix reflect offset">
+    <link name="${prefix}_caster_wheel">
+      <inertial>
+        <origin xyz="0 0 0" rpy="0 0 0"/>
+        <mass value="0.5"/>
+        <xacro:sphere_inertia m="0.5" r="${caster_radius}"/>
+      </inertial>
+      <visual>
+        <origin xyz="0 0 0" rpy="0 0 0"/>
+        <geometry>
+          <sphere radius="${caster_radius}"/>
+        </geometry>
+        <material name="caster_material">
+          <color rgba="0.29804 0.29804 0.29804 1"/>
+        </material>
+      </visual>
+      <collision>
+        <origin xyz="0 0 0" rpy="0 0 0"/>
+        <geometry>
+          <sphere radius="${caster_radius}"/>
+        </geometry>
+      </collision>
+    </link>
+    <joint name="${prefix}_caster_wheel_joint" type="continuous">
+      <origin xyz="${caster_x * offset} ${caster_y * reflect} ${caster_z}" rpy="0 0 0"/>
+      <parent link="chassibigga"/>
+      <child link="${prefix}_caster_wheel"/>
+      <axis xyz="0 1 0"/>
+      <dynamics damping="0.5" friction="0.5"/>
+    </joint>
+  </xacro:macro>
+  <xacro:caster_wheel prefix="front_left" reflect="1" offset="1" />
+  <xacro:caster_wheel prefix="front_right" reflect="-1" offset="1" />
+  <xacro:caster_wheel prefix="rear_left" reflect="1" offset="-1" />
+  <xacro:caster_wheel prefix="rear_right" reflect="-1" offset="-1" />
   <!-- Hitch point at the back of tugger -->
   <link name="hitch_link">
@@ -143,5 +200,5 @@
   </link>
   <joint name="hitch_joint" type="fixed">
-    <origin xyz="0 0.35 0.14260" rpy="0 0 0"/>
+    <origin xyz="0 0.35 ${chassi_z + hitch_offset_z}" rpy="0 0 0"/>
     <parent link="chassibigga"/>
     <child link="hitch_link"/>
@@ -173,5 +230,5 @@
     <parent link="chassibigga"/>
     <child link="lidar_link"/>
-    <origin xyz="0 -0.25 0.34" rpy="0 0 0"/>
+    <origin xyz="0 -0.25 ${chassi_z + lidar_offset_z}" rpy="0 0 0"/>
   </joint>
 </robot>
